Commit message: add requirements.txt

File: temp1.urdf (robot description, URDF)
Before this commit: robot pepe, 12 links, 11 joints
Links:
- removed link 310
- removed link 311
- removed link 39
- added link 19, mass 6.281300540076709; collision cylinder length=1.9998 radius=0.9999; visual cylinder length=1.9998 radius=0.9999
- added link 210, mass 0.0637264246388024; collision cylinder length=1.8650633825301641 radius=0.10428888937644346; visual cylinder length=1.8650633825301641 radius=0.10428888937644346
- added link 211, mass 0.0637264246388024; collision cylinder length=1.8650633825301641 radius=0.10428888937644346; visual cylinder length=1.8650633825301641 radius=0.10428888937644346
- added link 212, mass 0.0637264246388024; collision cylinder length=1.8650633825301641 radius=0.10428888937644346; visual cylinder length=1.8650633825301641 radius=0.10428888937644346
- link 0: mass 0.15735352719442636 -> 0.0637264246388024; geometry collision cylinder length=1.8650633825301641 radius=0.10428888937644346; visual cylinder length=1.8650633825301641 radius=0.10428888937644346
- link 11: mass 4.467304882838585e-06 -> 6.281300540076709; geometry collision cylinder length=1.9998 radius=0.9999; visual cylinder length=1.9998 radius=0.9999
- link 15: mass 4.467304882838585e-06 -> 6.281300540076709; geometry collision cylinder length=1.9998 radius=0.9999; visual cylinder length=1.9998 radius=0.9999
- link 22: mass 0.9483313163545366 -> 0.0637264246388024; geometry collision cylinder length=1.8650633825301641 radius=0.10428888937644346; visual cylinder length=1.8650633825301641 radius=0.10428888937644346
- link 23: mass 0.9483313163545366 -> 0.0637264246388024; geometry collision cylinder length=1.8650633825301641 radius=0.10428888937644346; visual cylinder length=1.8650633825301641 radius=0.10428888937644346
- link 24: mass 0.9483313163545366 -> 0.0637264246388024; geometry collision cylinder length=1.8650633825301641 radius=0.10428888937644346; visual cylinder length=1.8650633825301641 radius=0.10428888937644346
- link 26: mass 0.9483313163545366 -> 0.0637264246388024; geometry collision cylinder length=1.8650633825301641 radius=0.10428888937644346; visual cylinder length=1.8650633825301641 radius=0.10428888937644346
- link 27: mass 0.9483313163545366 -> 0.0637264246388024; geometry collision cylinder length=1.8650633825301641 radius=0.10428888937644346; visual cylinder length=1.8650633825301641 radius=0.10428888937644346
- link 28: mass 0.9483313163545366 -> 0.0637264246388024; geometry collision cylinder length=1.8650633825301641 radius=0.10428888937644346; visual cylinder length=1.8650633825301641 radius=0.10428888937644346
Joints:
- removed joint 310_to_0
- removed joint 311_to_0
- removed joint 39_to_0
- added joint 19_to_0: type revolute, parent 0, child 19, origin xyz=0.9999 0.9999 0.9999 rpy=25.130227954595473 6.282556988648868 6.282556988648868, axis 0 0 1, limit lower=3.1415 upper=-3.1415 effort=1 velocity=1
- added joint 210_to_19: type revolute, parent 19, child 210, origin xyz=0.8963054758440083 0.9999 0.9999 rpy=12.565113977297736 6.282556988648868 6.282556988648868, axis 0 0 1, limit lower=3.1415 upper=-3.1415 effort=1 velocity=1
- added joint 211_to_19: type revolute, parent 19, child 211, origin xyz=0.8963054758440083 0.9999 0.9999 rpy=18.847670965946605 6.282556988648868 6.282556988648868, axis 0 0 1, limit lower=3.1415 upper=-3.1415 effort=1 velocity=1
- added joint 212_to_19: type revolute, parent 19, child 212, origin xyz=0.8963054758440083 0.9999 0.9999 rpy=25.130227954595473 6.282556988648868 6.282556988648868, axis 0 0 1, limit lower=3.1415 upper=-3.1415 effort=1 velocity=1
- joint 11_to_0: axis 0 1 0 -> 0 0 1; origin xyz=0.7236069504422373 0.9885880704038275 0.4161850445130292 rpy=4.853035674087351 6.262356433276231 4.280533725595206 -> xyz=0.9999 0.9999 0.9999 rpy=12.565113977297736 6.282556988648868 6.282556988648868
- joint 15_to_0: axis 0 1 0 -> 0 0 1; origin xyz=0.7236069504422373 0.9885880704038275 0.4161850445130292 rpy=7.2795535111310254 6.262356433276231 4.280533725595206 -> xyz=0.9999 0.9999 0.9999 rpy=18.847670965946605 6.282556988648868 6.282556988648868
- joint 22_to_11: axis 0 1 0 -> 0 0 1; origin xyz=0.9665428940687371 0.9896372884871573 0.8568418066111094 rpy=0.12511119359624798 5.869302657479386 3.7471401696628437 -> xyz=0.8963054758440083 0.9999 0.9999 rpy=12.565113977297736 6.282556988648868 6.282556988648868
- joint 23_to_11: axis 0 1 0 -> 0 0 1; origin xyz=0.9665428940687371 0.9896372884871573 0.8568418066111094 rpy=0.18766679039437195 5.869302657479386 3.7471401696628437 -> xyz=0.8963054758440083 0.9999 0.9999 rpy=18.847670965946605 6.282556988648868 6.282556988648868
- joint 24_to_11: axis 0 1 0 -> 0 0 1; origin xyz=0.9665428940687371 0.9896372884871573 0.8568418066111094 rpy=0.25022238719249595 5.869302657479386 3.7471401696628437 -> xyz=0.8963054758440083 0.9999 0.9999 rpy=25.130227954595473 6.282556988648868 6.282556988648868
- joint 26_to_15: axis 0 1 0 -> 0 0 1; origin xyz=0.9665428940687371 0.9896372884871573 0.8568418066111094 rpy=0.12511119359624798 5.869302657479386 3.7471401696628437 -> xyz=0.8963054758440083 0.9999 0.9999 rpy=12.565113977297736 6.282556988648868 6.282556988648868
- joint 27_to_15: axis 0 1 0 -> 0 0 1; origin xyz=0.9665428940687371 0.9896372884871573 0.8568418066111094 rpy=0.18766679039437195 5.869302657479386 3.7471401696628437 -> xyz=0.8963054758440083 0.9999 0.9999 rpy=18.847670965946605 6.282556988648868 6.282556988648868
- joint 28_to_15: axis 0 1 0 -> 0 0 1; origin xyz=0.9665428940687371 0.9896372884871573 0.8568418066111094 rpy=0.25022238719249595 5.869302657479386 3.7471401696628437 -> xyz=0.8963054758440083 0.9999 0.9999 rpy=25.130227954595473 6.282556988648868 6.282556988648868

File: temp10.urdf (robot description, URDF)
Before this commit: robot pepe, 13 links, 12 joints
Links:
- link 210: mass 6.281300540076709 -> 0.00019415638996012175; geometry collision cylinder length=0.20469765564289283 radius=0.01737578657019445; visual cylinder length=0.20469765564289283 radius=0.01737578657019445
- link 211: mass 6.281300540076709 -> 0.00019415638996012175; geometry collision cylinder length=0.20469765564289283 radius=0.01737578657019445; visual cylinder length=0.20469765564289283 radius=0.01737578657019445
- link 212: mass 6.281300540076709 -> 0.00019415638996012175; geometry collision cylinder length=0.20469765564289283 radius=0.01737578657019445; visual cylinder length=0.20469765564289283 radius=0.01737578657019445
- link 22: mass 6.281300540076709 -> 0.00019415638996012175; geometry collision cylinder length=0.20469765564289283 radius=0.01737578657019445; visual cylinder length=0.20469765564289283 radius=0.01737578657019445
- link 23: mass 6.281300540076709 -> 0.00019415638996012175; geometry collision cylinder length=0.20469765564289283 radius=0.01737578657019445; visual cylinder length=0.20469765564289283 radius=0.01737578657019445
- link 24: mass 6.281300540076709 -> 0.00019415638996012175; geometry collision cylinder length=0.20469765564289283 radius=0.01737578657019445; visual cylinder length=0.20469765564289283 radius=0.01737578657019445
- link 26: mass 6.281300540076709 -> 0.00019415638996012175; geometry collision cylinder length=0.20469765564289283 radius=0.01737578657019445; visual cylinder length=0.20469765564289283 radius=0.01737578657019445
- link 27: mass 6.281300540076709 -> 0.00019415638996012175; geometry collision cylinder length=0.20469765564289283 radius=0.01737578657019445; visual cylinder length=0.20469765564289283 radius=0.01737578657019445
- link 28: mass 6.281300540076709 -> 0.00019415638996012175; geometry collision cylinder length=0.20469765564289283 radius=0.01737578657019445; visual cylinder length=0.20469765564289283 radius=0.01737578657019445

File: temp11.urdf (robot description, URDF)
Before this commit: robot pepe, 4 links, 3 joints
Links:
- link 0: mass 0.06833017321898761 -> 0.0637264246388024; geometry collision cylinder length=1.8650633825301641 radius=0.10428888937644346; visual cylinder length=1.8650633825301641 radius=0.10428888937644346

File: temp2.urdf (robot description, URDF)
Before this commit: robot pepe, 1 links, 0 joints
Links:
- added link 11, mass 0.0637264246388024; collision cylinder length=1.8650633825301641 radius=0.10428888937644346; visual cylinder length=1.8650633825301641 radius=0.10428888937644346
- added link 12, mass 0.0637264246388024; collision cylinder length=1.8650633825301641 radius=0.10428888937644346; visual cylinder length=1.8650633825301641 radius=0.10428888937644346
- added link 13, mass 0.0637264246388024; collision cylinder length=1.8650633825301641 radius=0.10428888937644346; visual cylinder length=1.8650633825301641 radius=0.10428888937644346
- link 0: mass 0.19742596388519396 -> 0.00019415638996012175; geometry collision cylinder length=0.20469765564289283 radius=0.01737578657019445; visual cylinder length=0.20469765564289283 radius=0.01737578657019445
Joints:
- added joint 11_to_0: type revolute, parent 0, child 11, origin xyz=0.9963054758440083 0.9999 0.9999 rpy=12.565113977297736 6.282556988648868 6.282556988648868, axis 0 0 1, limit lower=3.1415 upper=-3.1415 effort=1 velocity=1
- added joint 12_to_0: type revolute, parent 0, child 12, origin xyz=0.9963054758440083 0.9999 0.9999 rpy=18.847670965946605 6.282556988648868 6.282556988648868, axis 0 0 1, limit lower=3.1415 upper=-3.1415 effort=1 velocity=1
- added joint 13_to_0: type revolute, parent 0, child 13, origin xyz=0.9963054758440083 0.9999 0.9999 rpy=25.130227954595473 6.282556988648868 6.282556988648868, axis 0 0 1, limit lower=3.1415 upper=-3.1415 effort=1 velocity=1

File: temp3.urdf (robot description, URDF)
Before this commit: robot pepe, 15 links, 14 joints
Links:
- removed link 18
- removed link 212
- removed link 22
- removed link 25
- removed link 29
- removed link 310
- removed link 311
- removed link 313
- removed link 314
- removed link 33
- removed link 34
- removed link 36
- removed link 37
- added link 12, mass 6.281300540076709; collision cylinder length=1.9998 radius=0.9999; visual cylinder length=1.9998 radius=0.9999
- added link 13, mass 6.281300540076709; collision cylinder length=1.9998 radius=0.9999; visual cylinder length=1.9998 radius=0.9999
- link 0: mass 1.0360342360436707 -> 6.281300540076709; geometry collision cylinder length=1.9998 radius=0.9999; visual cylinder length=1.9998 radius=0.9999
- link 11: mass 4.467304882838585e-06 -> 6.281300540076709; geometry collision cylinder length=1.9998 radius=0.9999; visual cylinder length=1.9998 radius=0.9999
Joints:
- removed joint 18_to_0
- removed joint 212_to_18
- removed joint 22_to_11
- removed joint 25_to_11
- removed joint 29_to_18
- removed joint 310_to_29
- removed joint 311_to_29
- removed joint 313_to_212
- removed joint 314_to_212
- removed joint 33_to_22
- removed joint 34_to_22
- removed joint 36_to_25
- removed joint 37_to_25
- added joint 12_to_0: type revolute, parent 0, child 12, origin xyz=0.9999 0.9999 0.9999 rpy=18.847670965946605 6.282556988648868 6.282556988648868, axis 0 0 1, limit lower=3.1415 upper=-3.1415 effort=1 velocity=1
- added joint 13_to_0: type revolute, parent 0, child 13, origin xyz=0.9999 0.9999 0.9999 rpy=25.130227954595473 6.282556988648868 6.282556988648868, axis 0 0 1, limit lower=3.1415 upper=-3.1415 effort=1 velocity=1
- joint 11_to_0: axis 0 1 0 -> 0 0 1; origin xyz=0.7236069504422373 0.9999 0.4161850445130292 rpy=3.596398612651434 6.262356433276231 4.280533725595206 -> xyz=0.9999 0.9999 0.9999 rpy=12.565113977297736 6.282556988648868 6.282556988648868

File: temp4.urdf (robot description, URDF)
Before this commit: robot pepe, 2 links, 1 joints
Links:
- added link 12, mass 0.00019415638996012175; collision cylinder length=0.20469765564289283 radius=0.01737578657019445; visual cylinder length=0.20469765564289283 radius=0.01737578657019445
- added link 23, mass 0.41984121088199017; collision cylinder length=1.1619374222954129 radius=0.33913782223713174; visual cylinder length=1.1619374222954129 radius=0.33913782223713174
- link 0: mass 1.0360342360436707 -> 6.281300540076709; geometry collision cylinder length=1.9998 radius=0.9999; visual cylinder length=1.9998 radius=0.9999
- link 11: mass 0.3066418042690306 -> 0.00019415638996012175; geometry collision cylinder length=0.20469765564289283 radius=0.01737578657019445; visual cylinder length=0.20469765564289283 radius=0.01737578657019445
Joints:
- added joint 12_to_0: type revolute, parent 0, child 12, origin xyz=0.9999 0.9999 0.9999 rpy=18.847670965946605 6.282556988648868 6.282556988648868, axis 0 0 1, limit lower=3.1415 upper=-3.1415 effort=1 velocity=1
- added joint 23_to_0: type revolute, parent 0, child 23, origin xyz=0.8168537846017668 0.4317745097967489 0.8178267908170648 rpy=3.7543803664084434 1.5707369796363668 4.489869818886058, axis 0 0 1, limit lower=3.1415 upper=-3.1415 effort=1 velocity=1
- joint 11_to_0: origin xyz=0.43638400265132093 0.035632360108815986 0.31232581489814226 rpy=11.059927898506901 2.536670462446014 1.6217615205138476 -> xyz=0.9999 0.9999 0.9999 rpy=12.565113977297736 6.282556988648868 6.282556988648868

File: temp6.urdf (robot description, URDF)
Before this commit: robot pepe, 2 links, 1 joints
Links:
- added link 15, mass 0.0637264246388024; collision cylinder length=1.8650633825301641 radius=0.10428888937644346; visual cylinder length=1.8650633825301641 radius=0.10428888937644346
- added link 19, mass 0.0637264246388024; collision cylinder length=1.8650633825301641 radius=0.10428888937644346; visual cylinder length=1.8650633825301641 radius=0.10428888937644346
- added link 210, mass 6.281300540076709; collision cylinder length=1.9998 radius=0.9999; visual cylinder length=1.9998 radius=0.9999
- added link 211, mass 6.281300540076709; collision cylinder length=1.9998 radius=0.9999; visual cylinder length=1.9998 radius=0.9999
- added link 212, mass 6.281300540076709; collision cylinder length=1.9998 radius=0.9999; visual cylinder length=1.9998 radius=0.9999
- added link 22, mass 6.281300540076709; collision cylinder length=1.9998 radius=0.9999; visual cylinder length=1.9998 radius=0.9999
- added link 23, mass 6.281300540076709; collision cylinder length=1.9998 radius=0.9999; visual cylinder length=1.9998 radius=0.9999
- added link 24, mass 6.281300540076709; collision cylinder length=1.9998 radius=0.9999; visual cylinder length=1.9998 radius=0.9999
- added link 26, mass 6.281300540076709; collision cylinder length=1.9998 radius=0.9999; visual cylinder length=1.9998 radius=0.9999
- added link 27, mass 6.281300540076709; collision cylinder length=1.9998 radius=0.9999; visual cylinder length=1.9998 radius=0.9999
- added link 28, mass 6.281300540076709; collision cylinder length=1.9998 radius=0.9999; visual cylinder length=1.9998 radius=0.9999
- link 0: mass 0.5560741273262054 -> 0.00019415638996012175; geometry collision cylinder length=0.20469765564289283 radius=0.01737578657019445; visual cylinder length=0.20469765564289283 radius=0.01737578657019445
- link 11: mass 0.3066418042690306 -> 0.0637264246388024; geometry collision cylinder length=1.8650633825301641 radius=0.10428888937644346; visual cylinder length=1.8650633825301641 radius=0.10428888937644346
Joints:
- added joint 15_to_0: type revolute, parent 0, child 15, origin xyz=0.8963054758440083 0.9999 0.9999 rpy=18.847670965946605 6.282556988648868 6.282556988648868, axis 0 0 1, limit lower=3.1415 upper=-3.1415 effort=1 velocity=1
- added joint 19_to_0: type revolute, parent 0, child 19, origin xyz=0.8963054758440083 0.9999 0.9999 rpy=25.130227954595473 6.282556988648868 6.282556988648868, axis 0 0 1, limit lower=3.1415 upper=-3.1415 effort=1 velocity=1
- added joint 210_to_19: type revolute, parent 19, child 210, origin xyz=0.9999 0.9999 0.9999 rpy=12.565113977297736 6.282556988648868 6.282556988648868, axis 0 0 1, limit lower=3.1415 upper=-3.1415 effort=1 velocity=1
- added joint 211_to_19: type revolute, parent 19, child 211, origin xyz=0.9999 0.9999 0.9999 rpy=18.847670965946605 6.282556988648868 6.282556988648868, axis 0 0 1, limit lower=3.1415 upper=-3.1415 effort=1 velocity=1
- added joint 212_to_19: type revolute, parent 19, child 212, origin xyz=0.9999 0.9999 0.9999 rpy=25.130227954595473 6.282556988648868 6.282556988648868, axis 0 0 1, limit lower=3.1415 upper=-3.1415 effort=1 velocity=1
- added joint 22_to_11: type revolute, parent 11, child 22, origin xyz=0.9999 0.9999 0.9999 rpy=12.565113977297736 6.282556988648868 6.282556988648868, axis 0 0 1, limit lower=3.1415 upper=-3.1415 effort=1 velocity=1
- added joint 23_to_11: type revolute, parent 11, child 23, origin xyz=0.9999 0.9999 0.9999 rpy=18.847670965946605 6.282556988648868 6.282556988648868, axis 0 0 1, limit lower=3.1415 upper=-3.1415 effort=1 velocity=1
- added joint 24_to_11: type revolute, parent 11, child 24, origin xyz=0.9999 0.9999 0.9999 rpy=25.130227954595473 6.282556988648868 6.282556988648868, axis 0 0 1, limit lower=3.1415 upper=-3.1415 effort=1 velocity=1
- added joint 26_to_15: type revolute, parent 15, child 26, origin xyz=0.9999 0.9999 0.9999 rpy=12.565113977297736 6.282556988648868 6.282556988648868, axis 0 0 1, limit lower=3.1415 upper=-3.1415 effort=1 velocity=1
- added joint 27_to_15: type revolute, parent 15, child 27, origin xyz=0.9999 0.9999 0.9999 rpy=18.847670965946605 6.282556988648868 6.282556988648868, axis 0 0 1, limit lower=3.1415 upper=-3.1415 effort=1 velocity=1
- added joint 28_to_15: type revolute, parent 15, child 28, origin xyz=0.9999 0.9999 0.9999 rpy=25.130227954595473 6.282556988648868 6.282556988648868, axis 0 0 1, limit lower=3.1415 upper=-3.1415 effort=1 velocity=1
- joint 11_to_0: origin xyz=0.33638400265132096 0.035632360108815986 0.41232581489814224 rpy=12.316564959942818 2.536670462446014 2.250080051231806 -> xyz=0.8963054758440083 0.9999 0.9999 rpy=12.565113977297736 6.282556988648868 6.282556988648868

File: temp7.urdf (robot description, URDF)
Before this commit: robot pepe, 4 links, 3 joints
Links:
- removed link 11
- removed link 22
- removed link 23
- link 0: mass 0.018782858160138177 -> 6.281300540076709; geometry collision cylinder length=1.9998 radius=0.9999; visual cylinder length=1.9998 radius=0.9999
Joints:
- removed joint 11_to_0
- removed joint 22_to_0
- removed joint 23_to_0

File: temp8.urdf (robot description, URDF)
Before this commit: robot pepe, 5 links, 4 joints
Links:
- added link 15, mass 0.0637264246388024; collision cylinder length=1.8650633825301641 radius=0.10428888937644346; visual cylinder length=1.8650633825301641 radius=0.10428888937644346
- added link 19, mass 0.0637264246388024; collision cylinder length=1.8650633825301641 radius=0.10428888937644346; visual cylinder length=1.8650633825301641 radius=0.10428888937644346
- added link 210, mass 6.281300540076709; collision cylinder length=1.9998 radius=0.9999; visual cylinder length=1.9998 radius=0.9999
- added link 211, mass 6.281300540076709; collision cylinder length=1.9998 radius=0.9999; visual cylinder length=1.9998 radius=0.9999
- added link 212, mass 6.281300540076709; collision cylinder length=1.9998 radius=0.9999; visual cylinder length=1.9998 radius=0.9999
- added link 26, mass 6.281300540076709; collision cylinder length=1.9998 radius=0.9999; visual cylinder length=1.9998 radius=0.9999
- added link 27, mass 6.281300540076709; collision cylinder length=1.9998 radius=0.9999; visual cylinder length=1.9998 radius=0.9999
- added link 28, mass 6.281300540076709; collision cylinder length=1.9998 radius=0.9999; visual cylinder length=1.9998 radius=0.9999
- link 0: mass 1.4176451191353034 -> 0.00019415638996012175; geometry collision cylinder length=0.20469765564289283 radius=0.01737578657019445; visual cylinder length=0.20469765564289283 radius=0.01737578657019445
- link 11: mass 0.08825492213118463 -> 0.0637264246388024; geometry collision cylinder length=1.8650633825301641 radius=0.10428888937644346; visual cylinder length=1.8650633825301641 radius=0.10428888937644346
- link 22: mass 1.4176451191353034 -> 6.281300540076709; geometry collision cylinder length=1.9998 radius=0.9999; visual cylinder length=1.9998 radius=0.9999
- link 23: mass 1.4176451191353034 -> 6.281300540076709; geometry collision cylinder length=1.9998 radius=0.9999; visual cylinder length=1.9998 radius=0.9999
- link 24: mass 1.4176451191353034 -> 6.281300540076709; geometry collision cylinder length=1.9998 radius=0.9999; visual cylinder length=1.9998 radius=0.9999
Joints:
- removed joint 22_to_0
- removed joint 23_to_0
- removed joint 24_to_0
- added joint 15_to_0: type revolute, parent 0, child 15, origin xyz=0.8963054758440083 0.9999 0.9999 rpy=18.847670965946605 6.282556988648868 6.282556988648868, axis 0 0 1, limit lower=3.1415 upper=-3.1415 effort=1 velocity=1
- added joint 19_to_0: type revolute, parent 0, child 19, origin xyz=0.8963054758440083 0.9999 0.9999 rpy=25.130227954595473 6.282556988648868 6.282556988648868, axis 0 0 1, limit lower=3.1415 upper=-3.1415 effort=1 velocity=1
- added joint 210_to_19: type revolute, parent 19, child 210, origin xyz=0.9999 0.9999 0.9999 rpy=12.565113977297736 6.282556988648868 6.282556988648868, axis 0 0 1, limit lower=3.1415 upper=-3.1415 effort=1 velocity=1
- added joint 211_to_19: type revolute, parent 19, child 211, origin xyz=0.9999 0.9999 0.9999 rpy=18.847670965946605 6.282556988648868 6.282556988648868, axis 0 0 1, limit lower=3.1415 upper=-3.1415 effort=1 velocity=1
- added joint 212_to_19: type revolute, parent 19, child 212, origin xyz=0.9999 0.9999 0.9999 rpy=25.130227954595473 6.282556988648868 6.282556988648868, axis 0 0 1, limit lower=3.1415 upper=-3.1415 effort=1 velocity=1
- added joint 22_to_11: type revolute, parent 11, child 22, origin xyz=0.9999 0.9999 0.9999 rpy=12.565113977297736 6.282556988648868 6.282556988648868, axis 0 0 1, limit lower=3.1415 upper=-3.1415 effort=1 velocity=1
- added joint 23_to_11: type revolute, parent 11, child 23, origin xyz=0.9999 0.9999 0.9999 rpy=18.847670965946605 6.282556988648868 6.282556988648868, axis 0 0 1, limit lower=3.1415 upper=-3.1415 effort=1 velocity=1
- added joint 24_to_11: type revolute, parent 11, child 24, origin xyz=0.9999 0.9999 0.9999 rpy=25.130227954595473 6.282556988648868 6.282556988648868, axis 0 0 1, limit lower=3.1415 upper=-3.1415 effort=1 velocity=1
- added joint 26_to_15: type revolute, parent 15, child 26, origin xyz=0.9999 0.9999 0.9999 rpy=12.565113977297736 6.282556988648868 6.282556988648868, axis 0 0 1, limit lower=3.1415 upper=-3.1415 effort=1 velocity=1
- added joint 27_to_15: type revolute, parent 15, child 27, origin xyz=0.9999 0.9999 0.9999 rpy=18.847670965946605 6.282556988648868 6.282556988648868, axis 0 0 1, limit lower=3.1415 upper=-3.1415 effort=1 velocity=1
- added joint 28_to_15: type revolute, parent 15, child 28, origin xyz=0.9999 0.9999 0.9999 rpy=25.130227954595473 6.282556988648868 6.282556988648868, axis 0 0 1, limit lower=3.1415 upper=-3.1415 effort=1 velocity=1
- joint 11_to_0: origin xyz=0.20275605527502139 0.9999 0.2447046369169771 rpy=0.9411766697284422 6.282556988648868 4.669752477075483 -> xyz=0.8963054758440083 0.9999 0.9999 rpy=12.565113977297736 6.282556988648868 6.282556988648868
