Commit message: add requirements.txt

File: temp9.urdf (robot description, URDF)
Before this commit: robot pepe, 4 links, 3 joints
Links:
- removed link 12
- removed link 13
- added link 15, mass 0.0637264246388024; collision cylinder length=1.8650633825301641 radius=0.10428888937644346; visual cylinder length=1.8650633825301641 radius=0.10428888937644346
- added link 19, mass 0.0637264246388024; collision cylinder length=1.8650633825301641 radius=0.10428888937644346; visual cylinder length=1.8650633825301641 radius=0.10428888937644346
- added link 210, mass 6.281300540076709; collision cylinder length=1.9998 radius=0.9999; visual cylinder length=1.9998 radius=0.9999
- added link 211, mass 6.281300540076709; collision cylinder length=1.9998 radius=0.9999; visual cylinder length=1.9998 radius=0.9999
- added link 212, mass 6.281300540076709; collision cylinder length=1.9998 radius=0.9999; visual cylinder length=1.9998 radius=0.9999
- added link 22, mass 6.281300540076709; collision cylinder length=1.9998 radius=0.9999; visual cylinder length=1.9998 radius=0.9999
- added link 23, mass 6.281300540076709; collision cylinder length=1.9998 radius=0.9999; visual cylinder length=1.9998 radius=0.9999
- added link 24, mass 6.281300540076709; collision cylinder length=1.9998 radius=0.9999; visual cylinder length=1.9998 radius=0.9999
- added link 26, mass 6.281300540076709; collision cylinder length=1.9998 radius=0.9999; visual cylinder length=1.9998 radius=0.9999
- added link 27, mass 6.281300540076709; collision cylinder length=1.9998 radius=0.9999; visual cylinder length=1.9998 radius=0.9999
- added link 28, mass 6.281300540076709; collision cylinder length=1.9998 radius=0.9999; visual cylinder length=1.9998 radius=0.9999
- link 0: mass 1.4625210014394228 -> 6.281300540076709; geometry collision cylinder length=1.9998 radius=0.9999; visual cylinder length=1.9998 radius=0.9999
- link 11: mass 0.12978270156493504 -> 0.0637264246388024; geometry collision cylinder length=1.8650633825301641 radius=0.10428888937644346; visual cylinder length=1.8650633825301641 radius=0.10428888937644346
Joints:
- removed joint 12_to_0
- removed joint 13_to_0
- added joint 15_to_0: type revolute, parent 0, child 15, origin xyz=0.8963054758440083 0.9999 0.9999 rpy=18.847670965946605 6.282556988648868 6.282556988648868, axis 0 0 1, limit lower=3.1415 upper=-3.1415 effort=1 velocity=1
- added joint 19_to_0: type revolute, parent 0, child 19, origin xyz=0.8963054758440083 0.9999 0.9999 rpy=25.130227954595473 6.282556988648868 6.282556988648868, axis 0 0 1, limit lower=3.1415 upper=-3.1415 effort=1 velocity=1
- added joint 210_to_19: type revolute, parent 19, child 210, origin xyz=0.9999 0.9999 0.9999 rpy=12.565113977297736 6.282556988648868 6.282556988648868, axis 0 0 1, limit lower=3.1415 upper=-3.1415 effort=1 velocity=1
- added joint 211_to_19: type revolute, parent 19, child 211, origin xyz=0.9999 0.9999 0.9999 rpy=18.847670965946605 6.282556988648868 6.282556988648868, axis 0 0 1, limit lower=3.1415 upper=-3.1415 effort=1 velocity=1
- added joint 212_to_19: type revolute, parent 19, child 212, origin xyz=0.9999 0.9999 0.9999 rpy=25.130227954595473 6.282556988648868 6.282556988648868, axis 0 0 1, limit lower=3.1415 upper=-3.1415 effort=1 velocity=1
- added joint 22_to_11: type revolute, parent 11, child 22, origin xyz=0.9999 0.9999 0.9999 rpy=12.565113977297736 6.282556988648868 6.282556988648868, axis 0 0 1, limit lower=3.1415 upper=-3.1415 effort=1 velocity=1
- added joint 23_to_11: type revolute, parent 11, child 23, origin xyz=0.9999 0.9999 0.9999 rpy=18.847670965946605 6.282556988648868 6.282556988648868, axis 0 0 1, limit lower=3.1415 upper=-3.1415 effort=1 velocity=1
- added joint 24_to_11: type revolute, parent 11, child 24, origin xyz=0.9999 0.9999 0.9999 rpy=25.130227954595473 6.282556988648868 6.282556988648868, axis 0 0 1, limit lower=3.1415 upper=-3.1415 effort=1 velocity=1
- added joint 26_to_15: type revolute, parent 15, child 26, origin xyz=0.9999 0.9999 0.9999 rpy=12.565113977297736 6.282556988648868 6.282556988648868, axis 0 0 1, limit lower=3.1415 upper=-3.1415 effort=1 velocity=1
- added joint 27_to_15: type revolute, parent 15, child 27, origin xyz=0.9999 0.9999 0.9999 rpy=18.847670965946605 6.282556988648868 6.282556988648868, axis 0 0 1, limit lower=3.1415 upper=-3.1415 effort=1 velocity=1
- added joint 28_to_15: type revolute, parent 15, child 28, origin xyz=0.9999 0.9999 0.9999 rpy=25.130227954595473 6.282556988648868 6.282556988648868, axis 0 0 1, limit lower=3.1415 upper=-3.1415 effort=1 velocity=1
- joint 11_to_0: axis 1 0 0 -> 0 0 1; origin xyz=0.18457565513068275 0.37313347329975777 0.8217667791091414 rpy=6.524330174264022 4.717985807462383 2.359086977962126 -> xyz=0.8963054758440083 0.9999 0.9999 rpy=12.565113977297736 6.282556988648868 6.282556988648868
