Commit message: hyperparam search framework ready and 3 tests passing

File: temp0.urdf (robot description, URDF)
Before this commit: robot pepe, 10 links, 9 joints
Links:
- removed link 14
- removed link 17
- removed link 22
- removed link 23
- removed link 25
- removed link 26
- removed link 28
- removed link 29
- added link 12, mass 0.605610648863151; collision cylinder length=1.848696671994538 radius=0.32291556970490987; visual cylinder length=1.848696671994538 radius=0.32291556970490987
- added link 13, mass 0.605610648863151; collision cylinder length=1.848696671994538 radius=0.32291556970490987; visual cylinder length=1.848696671994538 radius=0.32291556970490987
- link 0: mass 0.02321125271215263 -> 0.32333990492988784; geometry collision cylinder length=0.1840588742756495 radius=0.7477842884599845; visual cylinder length=0.1840588742756495 radius=0.7477842884599845
- link 11: mass 0.12978270156493504 -> 0.605610648863151; geometry collision cylinder length=1.848696671994538 radius=0.32291556970490987; visual cylinder length=1.848696671994538 radius=0.32291556970490987
Joints:
- removed joint 14_to_0
- removed joint 17_to_0
- removed joint 22_to_11
- removed joint 23_to_11
- removed joint 25_to_14
- removed joint 26_to_14
- removed joint 28_to_17
- removed joint 29_to_17
- added joint 12_to_0: type revolute, parent 0, child 12, origin xyz=0.9347096686071067 0.9999 0.6316106344170129 rpy=18.847670965946605 6.282556988648868 4.105571388352411, axis 0 0 1, limit lower=3.1415 upper=-3.1415 effort=1 velocity=1
- added joint 13_to_0: type revolute, parent 0, child 13, origin xyz=0.9347096686071067 0.9999 0.6316106344170129 rpy=25.130227954595473 6.282556988648868 4.105571388352411, axis 0 0 1, limit lower=3.1415 upper=-3.1415 effort=1 velocity=1
- joint 11_to_0: axis 1 0 0 -> 0 0 1; origin xyz=0.18457565513068275 0.37313347329975777 0.7217667791091414 rpy=6.524330174264022 4.717985807462383 2.359086977962126 -> xyz=0.9347096686071067 0.9999 0.6316106344170129 rpy=12.565113977297736 6.282556988648868 4.105571388352411

File: temp1.urdf (robot description, URDF)
Before this commit: robot pepe, 6 links, 5 joints
Links:
- removed link 12
- removed link 24
- added link 14, mass 3.012449546198092; collision cylinder length=0.9590842794497736 radius=0.9999; visual cylinder length=0.9590842794497736 radius=0.9999
- added link 22, mass 0.32333990492988784; collision cylinder length=0.1840588742756495 radius=0.7477842884599845; visual cylinder length=0.1840588742756495 radius=0.7477842884599845
- added link 26, mass 0.32333990492988784; collision cylinder length=0.1840588742756495 radius=0.7477842884599845; visual cylinder length=0.1840588742756495 radius=0.7477842884599845
- link 0: mass 1.0993942739023423 -> 0.32333990492988784; geometry collision cylinder length=0.1840588742756495 radius=0.7477842884599845; visual cylinder length=0.1840588742756495 radius=0.7477842884599845
- link 11: mass 1.4625210014394228 -> 3.012449546198092; geometry collision cylinder length=0.9590842794497736 radius=0.9999; visual cylinder length=0.9590842794497736 radius=0.9999
- link 23: mass 0.12978270156493504 -> 0.32333990492988784; geometry collision cylinder length=0.1840588742756495 radius=0.7477842884599845; visual cylinder length=0.1840588742756495 radius=0.7477842884599845
- link 25: mass 0.12978270156493504 -> 0.32333990492988784; geometry collision cylinder length=0.1840588742756495 radius=0.7477842884599845; visual cylinder length=0.1840588742756495 radius=0.7477842884599845
Joints:
- removed joint 12_to_0
- removed joint 23_to_0
- removed joint 24_to_0
- removed joint 25_to_0
- added joint 14_to_0: type revolute, parent 0, child 14, origin xyz=0.9999 0.9999 0.8113147983958526 rpy=2.5445954000779025 4.691213996647221 4.587332218059687, axis 1 0 0, limit lower=3.1415 upper=-3.1415 effort=1 velocity=1
- added joint 22_to_11: type revolute, parent 11, child 22, origin xyz=0.6468384730736209 0.3982034764994321 0.6535115948109418 rpy=6.60400922450185 5.6464283762735334 0.8638038636710728, axis 1 0 0, limit lower=3.1415 upper=-3.1415 effort=1 velocity=1
- added joint 23_to_11: type revolute, parent 11, child 23, origin xyz=0.6468384730736209 0.3982034764994321 0.6535115948109418 rpy=9.906013836752773 5.6464283762735334 0.8638038636710728, axis 1 0 0, limit lower=3.1415 upper=-3.1415 effort=1 velocity=1
- added joint 25_to_14: type revolute, parent 14, child 25, origin xyz=0.6468384730736209 0.3982034764994321 0.6535115948109418 rpy=6.60400922450185 5.6464283762735334 0.8638038636710728, axis 1 0 0, limit lower=3.1415 upper=-3.1415 effort=1 velocity=1
- added joint 26_to_14: type revolute, parent 14, child 26, origin xyz=0.6468384730736209 0.3982034764994321 0.6535115948109418 rpy=9.906013836752773 5.6464283762735334 0.8638038636710728, axis 1 0 0, limit lower=3.1415 upper=-3.1415 effort=1 velocity=1
- joint 11_to_0: axis 0 0 1 -> 1 0 0; origin xyz=0.6765749496532885 0.18662603572218528 0.22149339297314974 rpy=9.27380649927809 4.761254996217394 2.7830122907600003 -> xyz=0.9999 0.9999 0.8113147983958526 rpy=1.6963969333852684 4.691213996647221 4.587332218059687

File: temp2.urdf (robot description, URDF)
Before this commit: robot pepe, 6 links, 5 joints
Links:
- removed link 11
- removed link 12
- removed link 13
- removed link 24
- removed link 25
- link 0: mass 1.0383671212423773 -> 0.32333990492988784; geometry collision cylinder length=0.1840588742756495 radius=0.7477842884599845; visual cylinder length=0.1840588742756495 radius=0.7477842884599845
Joints:
- removed joint 11_to_0
- removed joint 12_to_0
- removed joint 13_to_0
- removed joint 24_to_0
- removed joint 25_to_0

File: temp3.urdf (robot description, URDF)
Before this commit: robot pepe, 7 links, 6 joints
Links:
- removed link 24
- removed link 25
- removed link 26
- link 0: mass 1.3664573012695778 -> 1.038778327639143; geometry collision cylinder length=1.848696671994538 radius=0.42291556970490984; visual cylinder length=1.848696671994538 radius=0.42291556970490984
- link 11: mass 0.1284845529504032 -> 0.048116617275910635; geometry collision cylinder length=0.05255946890700525 radius=0.5398177036498966; visual cylinder length=0.05255946890700525 radius=0.5398177036498966
- link 12: mass 0.1284845529504032 -> 0.048116617275910635; geometry collision cylinder length=0.05255946890700525 radius=0.5398177036498966; visual cylinder length=0.05255946890700525 radius=0.5398177036498966
- link 13: mass 0.1284845529504032 -> 0.048116617275910635; geometry collision cylinder length=0.05255946890700525 radius=0.5398177036498966; visual cylinder length=0.05255946890700525 radius=0.5398177036498966
Joints:
- removed joint 24_to_0
- removed joint 25_to_0
- removed joint 26_to_0
- joint 11_to_0: axis 1 0 0 -> 0 0 1; origin xyz=0.5955700154702805 0.7289445521847621 0.08632800227034598 rpy=1.6354206141385406 4.641392125360962 3.9820139839517577 -> xyz=0.5346921704194656 0.7675536365303309 0.03727917973075667 rpy=5.6612653984215715 3.1699043910322446 0.44175665736072767
- joint 12_to_0: axis 1 0 0 -> 0 0 1; origin xyz=0.5955700154702805 0.7289445521847621 0.08632800227034598 rpy=2.4531309212078107 4.641392125360962 3.9820139839517577 -> xyz=0.5346921704194656 0.7675536365303309 0.03727917973075667 rpy=8.491898097632358 3.1699043910322446 0.44175665736072767
- joint 13_to_0: axis 1 0 0 -> 0 0 1; origin xyz=0.5955700154702805 0.7289445521847621 0.08632800227034598 rpy=3.270841228277081 4.641392125360962 3.9820139839517577 -> xyz=0.5346921704194656 0.7675536365303309 0.03727917973075667 rpy=11.322530796843143 3.1699043910322446 0.44175665736072767

File: temp4.urdf (robot description, URDF)
Before this commit: robot pepe, 1 links, 0 joints
Links:
- link 0: mass 0.08825492213118463 -> 0.2886000077562378; geometry collision cylinder length=1.848696671994538 radius=0.22291556970490983; visual cylinder length=1.848696671994538 radius=0.22291556970490983

File: temp5.urdf (robot description, URDF)
Before this commit: robot pepe, 2 links, 1 joints
Links:
- added link 12, mass 0.32333990492988784; collision cylinder length=0.1840588742756495 radius=0.7477842884599845; visual cylinder length=0.1840588742756495 radius=0.7477842884599845
- added link 13, mass 0.32333990492988784; collision cylinder length=0.1840588742756495 radius=0.7477842884599845; visual cylinder length=0.1840588742756495 radius=0.7477842884599845
- added link 24, mass 0.05968430199862835; collision cylinder length=0.02449358809823976 radius=0.880701869373325; visual cylinder length=0.02449358809823976 radius=0.880701869373325
- added link 25, mass 0.05968430199862835; collision cylinder length=0.02449358809823976 radius=0.880701869373325; visual cylinder length=0.02449358809823976 radius=0.880701869373325
- added link 26, mass 0.05968430199862835; collision cylinder length=0.02449358809823976 radius=0.880701869373325; visual cylinder length=0.02449358809823976 radius=0.880701869373325
- link 0: mass 1.0993942739023423 -> 3.012449546198092; geometry collision cylinder length=0.9590842794497736 radius=0.9999; visual cylinder length=0.9590842794497736 radius=0.9999
- link 11: mass 0.08825492213118463 -> 0.32333990492988784; geometry collision cylinder length=0.1840588742756495 radius=0.7477842884599845; visual cylinder length=0.1840588742756495 radius=0.7477842884599845
Joints:
- added joint 12_to_0: type revolute, parent 0, child 12, origin xyz=0.6468384730736209 0.3982034764994321 0.6535115948109418 rpy=9.906013836752773 5.018109845555575 0.8638038636710728, axis 1 0 0, limit lower=3.1415 upper=-3.1415 effort=1 velocity=1
- added joint 13_to_0: type revolute, parent 0, child 13, origin xyz=0.6468384730736209 0.3982034764994321 0.6535115948109418 rpy=13.2080184490037 5.018109845555575 0.8638038636710728, axis 1 0 0, limit lower=3.1415 upper=-3.1415 effort=1 velocity=1
- added joint 24_to_0: type revolute, parent 0, child 24, origin xyz=0.623391653776098 0.4594726850384473 0.5002511972904059 rpy=13.404493168970667 2.197384708663479 1.0132440114302523, axis 0 0 1, limit lower=3.1415 upper=-3.1415 effort=1 velocity=1
- added joint 25_to_0: type revolute, parent 0, child 25, origin xyz=0.623391653776098 0.4594726850384473 0.5002511972904059 rpy=16.085391802764804 2.197384708663479 1.0132440114302523, axis 0 0 1, limit lower=3.1415 upper=-3.1415 effort=1 velocity=1
- added joint 26_to_0: type revolute, parent 0, child 26, origin xyz=0.623391653776098 0.4594726850384473 0.5002511972904059 rpy=18.766290436558936 2.197384708663479 1.0132440114302523, axis 0 0 1, limit lower=3.1415 upper=-3.1415 effort=1 velocity=1
- joint 11_to_0: axis 0 0 1 -> 1 0 0; origin xyz=0.20275605527502139 0.9999 0.1447046369169771 rpy=0.9411766697284422 5.990988104792695 4.041433946357524 -> xyz=0.6468384730736209 0.3982034764994321 0.6535115948109418 rpy=6.60400922450185 5.018109845555575 0.8638038636710728

File: temp6.urdf (robot description, URDF)
Before this commit: robot pepe, 5 links, 4 joints
Links:
- removed link 11
- removed link 13
- removed link 22
- removed link 24
- link 0: mass 1.0993942739023423 -> 0.32333990492988784; geometry collision cylinder length=0.1840588742756495 radius=0.7477842884599845; visual cylinder length=0.1840588742756495 radius=0.7477842884599845
Joints:
- removed joint 11_to_0
- removed joint 13_to_0
- removed joint 22_to_11
- removed joint 24_to_13

File: temp7.urdf (robot description, URDF)
Before this commit: robot pepe, 5 links, 4 joints
Links:
- removed link 12
- added link 15, mass 0.32333990492988784; collision cylinder length=0.1840588742756495 radius=0.7477842884599845; visual cylinder length=0.1840588742756495 radius=0.7477842884599845
- added link 19, mass 0.32333990492988784; collision cylinder length=0.1840588742756495 radius=0.7477842884599845; visual cylinder length=0.1840588742756495 radius=0.7477842884599845
- added link 210, mass 0.605610648863151; collision cylinder length=1.848696671994538 radius=0.32291556970490987; visual cylinder length=1.848696671994538 radius=0.32291556970490987
- added link 211, mass 0.605610648863151; collision cylinder length=1.848696671994538 radius=0.32291556970490987; visual cylinder length=1.848696671994538 radius=0.32291556970490987
- added link 212, mass 0.605610648863151; collision cylinder length=1.848696671994538 radius=0.32291556970490987; visual cylinder length=1.848696671994538 radius=0.32291556970490987
- added link 22, mass 0.605610648863151; collision cylinder length=1.848696671994538 radius=0.32291556970490987; visual cylinder length=1.848696671994538 radius=0.32291556970490987
- added link 26, mass 0.605610648863151; collision cylinder length=1.848696671994538 radius=0.32291556970490987; visual cylinder length=1.848696671994538 radius=0.32291556970490987
- added link 27, mass 0.605610648863151; collision cylinder length=1.848696671994538 radius=0.32291556970490987; visual cylinder length=1.848696671994538 radius=0.32291556970490987
- added link 28, mass 0.605610648863151; collision cylinder length=1.848696671994538 radius=0.32291556970490987; visual cylinder length=1.848696671994538 radius=0.32291556970490987
- link 0: mass 1.0993942739023423 -> 3.012449546198092; geometry collision cylinder length=0.9590842794497736 radius=0.9999; visual cylinder length=0.9590842794497736 radius=0.9999
- link 11: mass 1.0993942739023423 -> 0.32333990492988784; geometry collision cylinder length=0.1840588742756495 radius=0.7477842884599845; visual cylinder length=0.1840588742756495 radius=0.7477842884599845
- link 23: mass 2.023548893566616 -> 0.605610648863151; geometry collision cylinder length=1.848696671994538 radius=0.32291556970490987; visual cylinder length=1.848696671994538 radius=0.32291556970490987
- link 24: mass 2.023548893566616 -> 0.605610648863151; geometry collision cylinder length=1.848696671994538 radius=0.32291556970490987; visual cylinder length=1.848696671994538 radius=0.32291556970490987
Joints:
- removed joint 12_to_0
- removed joint 23_to_0
- removed joint 24_to_0
- added joint 15_to_0: type revolute, parent 0, child 15, origin xyz=0.6468384730736209 0.3982034764994321 0.6535115948109418 rpy=8.021058244598898 5.018109845555575 0.8638038636710728, axis 1 0 0, limit lower=3.1415 upper=-3.1415 effort=1 velocity=1
- added joint 19_to_0: type revolute, parent 0, child 19, origin xyz=0.6468384730736209 0.3982034764994321 0.6535115948109418 rpy=10.694744326131865 5.018109845555575 0.8638038636710728, axis 1 0 0, limit lower=3.1415 upper=-3.1415 effort=1 velocity=1
- added joint 210_to_19: type revolute, parent 19, child 210, origin xyz=0.8347096686071067 0.9999 0.7316106344170129 rpy=12.565113977297736 5.5907467448347274 4.105571388352411, axis 0 0 1, limit lower=3.1415 upper=-3.1415 effort=1 velocity=1
- added joint 211_to_19: type revolute, parent 19, child 211, origin xyz=0.8347096686071067 0.9999 0.7316106344170129 rpy=18.847670965946605 5.5907467448347274 4.105571388352411, axis 0 0 1, limit lower=3.1415 upper=-3.1415 effort=1 velocity=1
- added joint 212_to_19: type revolute, parent 19, child 212, origin xyz=0.8347096686071067 0.9999 0.7316106344170129 rpy=25.130227954595473 5.5907467448347274 4.105571388352411, axis 0 0 1, limit lower=3.1415 upper=-3.1415 effort=1 velocity=1
- added joint 22_to_11: type revolute, parent 11, child 22, origin xyz=0.8347096686071067 0.9999 0.7316106344170129 rpy=12.565113977297736 5.5907467448347274 4.105571388352411, axis 0 0 1, limit lower=3.1415 upper=-3.1415 effort=1 velocity=1
- added joint 23_to_11: type revolute, parent 11, child 23, origin xyz=0.8347096686071067 0.9999 0.7316106344170129 rpy=18.847670965946605 5.5907467448347274 4.105571388352411, axis 0 0 1, limit lower=3.1415 upper=-3.1415 effort=1 velocity=1
- added joint 24_to_11: type revolute, parent 11, child 24, origin xyz=0.8347096686071067 0.9999 0.7316106344170129 rpy=25.130227954595473 5.5907467448347274 4.105571388352411, axis 0 0 1, limit lower=3.1415 upper=-3.1415 effort=1 velocity=1
- added joint 26_to_15: type revolute, parent 15, child 26, origin xyz=0.8347096686071067 0.9999 0.7316106344170129 rpy=12.565113977297736 5.5907467448347274 4.105571388352411, axis 0 0 1, limit lower=3.1415 upper=-3.1415 effort=1 velocity=1
- added joint 27_to_15: type revolute, parent 15, child 27, origin xyz=0.8347096686071067 0.9999 0.7316106344170129 rpy=18.847670965946605 5.5907467448347274 4.105571388352411, axis 0 0 1, limit lower=3.1415 upper=-3.1415 effort=1 velocity=1
- added joint 28_to_15: type revolute, parent 15, child 28, origin xyz=0.8347096686071067 0.9999 0.7316106344170129 rpy=25.130227954595473 5.5907467448347274 4.105571388352411, axis 0 0 1, limit lower=3.1415 upper=-3.1415 effort=1 velocity=1
- joint 11_to_0: axis 0 1 0 -> 1 0 0; origin xyz=0.5765749496532885 0.18662603572218528 0.22149339297314974 rpy=10.530443560714005 4.761254996217394 2.7830122907600003 -> xyz=0.6468384730736209 0.3982034764994321 0.6535115948109418 rpy=5.347372163065932 5.018109845555575 0.8638038636710728
