Commit message: add retry mechanism upon exceptions

File: temp0.urdf (robot description, URDF)
Before this commit: robot pepe, 4 links, 3 joints
Links:
- removed link 12
- removed link 13
- link 0: mass 0.32333990492988784 -> 0.46696831044792275; geometry collision cylinder length=1.0481208226524537 radius=0.3765850662787882; visual cylinder length=1.0481208226524537 radius=0.3765850662787882
- link 11: mass 0.605610648863151 -> 0.19742596388519396; geometry collision cylinder length=0.9853454403519184 radius=0.2525416080782076; visual cylinder length=0.9853454403519184 radius=0.2525416080782076
Joints:
- removed joint 12_to_0
- removed joint 13_to_0
- joint 11_to_0: origin xyz=0.9347096686071067 0.9999 0.6316106344170129 rpy=12.565113977297736 6.282556988648868 4.105571388352411 -> xyz=0.33638400265132096 0.035632360108815986 0.41232581489814224 rpy=11.059927898506901 2.536670462446014 1.6217615205138476

File: temp1.urdf (robot description, URDF)
Before this commit: robot pepe, 7 links, 6 joints
Links:
- removed link 14
- removed link 25
- added link 15, mass 4.467304882838585e-06; collision cylinder length=1.9168577574955858 radius=0.0008612969648227331; visual cylinder length=1.9168577574955858 radius=0.0008612969648227331
- added link 24, mass 0.9483313163545366; collision cylinder length=1.8305118696539509 radius=0.40608676477427597; visual cylinder length=1.8305118696539509 radius=0.40608676477427597
- added link 27, mass 0.9483313163545366; collision cylinder length=1.8305118696539509 radius=0.40608676477427597; visual cylinder length=1.8305118696539509 radius=0.40608676477427597
- added link 28, mass 0.9483313163545366; collision cylinder length=1.8305118696539509 radius=0.40608676477427597; visual cylinder length=1.8305118696539509 radius=0.40608676477427597
- added link 310, mass 1.279194800911756; collision cylinder length=0.8778408121753121 radius=0.6810602327278827; visual cylinder length=0.8778408121753121 radius=0.6810602327278827
- added link 311, mass 1.279194800911756; collision cylinder length=0.8778408121753121 radius=0.6810602327278827; visual cylinder length=0.8778408121753121 radius=0.6810602327278827
- added link 39, mass 1.279194800911756; collision cylinder length=0.8778408121753121 radius=0.6810602327278827; visual cylinder length=0.8778408121753121 radius=0.6810602327278827
- link 0: mass 0.32333990492988784 -> 0.15735352719442636; geometry collision cylinder length=0.7853454403519184 radius=0.2525416080782076; visual cylinder length=0.7853454403519184 radius=0.2525416080782076
- link 11: mass 3.012449546198092 -> 4.467304882838585e-06; geometry collision cylinder length=1.9168577574955858 radius=0.0008612969648227331; visual cylinder length=1.9168577574955858 radius=0.0008612969648227331
- link 22: mass 0.32333990492988784 -> 0.9483313163545366; geometry collision cylinder length=1.8305118696539509 radius=0.40608676477427597; visual cylinder length=1.8305118696539509 radius=0.40608676477427597
- link 23: mass 0.32333990492988784 -> 0.9483313163545366; geometry collision cylinder length=1.8305118696539509 radius=0.40608676477427597; visual cylinder length=1.8305118696539509 radius=0.40608676477427597
- link 26: mass 0.32333990492988784 -> 0.9483313163545366; geometry collision cylinder length=1.8305118696539509 radius=0.40608676477427597; visual cylinder length=1.8305118696539509 radius=0.40608676477427597
Joints:
- removed joint 14_to_0
- removed joint 25_to_14
- removed joint 26_to_14
- added joint 15_to_0: type revolute, parent 0, child 15, origin xyz=0.7236069504422373 0.9885880704038275 0.4161850445130292 rpy=7.2795535111310254 6.262356433276231 4.280533725595206, axis 0 1 0, limit lower=3.1415 upper=-3.1415 effort=1 velocity=1
- added joint 24_to_11: type revolute, parent 11, child 24, origin xyz=0.9665428940687371 0.9896372884871573 0.8568418066111094 rpy=0.25022238719249595 5.869302657479386 3.7471401696628437, axis 0 1 0, limit lower=3.1415 upper=-3.1415 effort=1 velocity=1
- added joint 26_to_15: type revolute, parent 15, child 26, origin xyz=0.9665428940687371 0.9896372884871573 0.8568418066111094 rpy=0.12511119359624798 5.869302657479386 3.7471401696628437, axis 0 1 0, limit lower=3.1415 upper=-3.1415 effort=1 velocity=1
- added joint 27_to_15: type revolute, parent 15, child 27, origin xyz=0.9665428940687371 0.9896372884871573 0.8568418066111094 rpy=0.18766679039437195 5.869302657479386 3.7471401696628437, axis 0 1 0, limit lower=3.1415 upper=-3.1415 effort=1 velocity=1
- added joint 28_to_15: type revolute, parent 15, child 28, origin xyz=0.9665428940687371 0.9896372884871573 0.8568418066111094 rpy=0.25022238719249595 5.869302657479386 3.7471401696628437, axis 0 1 0, limit lower=3.1415 upper=-3.1415 effort=1 velocity=1
- added joint 310_to_0: type revolute, parent 0, child 310, origin xyz=0.912872583023103 0.511143821914881 0.06417149582715598 rpy=6.267350542972576 6.0545731271296654 1.7865608202423602, axis 1 0 0, limit lower=3.1415 upper=-3.1415 effort=1 velocity=1
- added joint 311_to_0: type revolute, parent 0, child 311, origin xyz=0.912872583023103 0.511143821914881 0.06417149582715598 rpy=7.5208206515670915 6.0545731271296654 1.7865608202423602, axis 1 0 0, limit lower=3.1415 upper=-3.1415 effort=1 velocity=1
- added joint 39_to_0: type revolute, parent 0, child 39, origin xyz=0.912872583023103 0.511143821914881 0.06417149582715598 rpy=5.013880434378061 6.0545731271296654 1.7865608202423602, axis 1 0 0, limit lower=3.1415 upper=-3.1415 effort=1 velocity=1
- joint 11_to_0: axis 1 0 0 -> 0 1 0; origin xyz=0.9999 0.9999 0.8113147983958526 rpy=1.6963969333852684 4.691213996647221 4.587332218059687 -> xyz=0.7236069504422373 0.9885880704038275 0.4161850445130292 rpy=4.853035674087351 6.262356433276231 4.280533725595206
- joint 22_to_11: axis 1 0 0 -> 0 1 0; origin xyz=0.6468384730736209 0.3982034764994321 0.6535115948109418 rpy=6.60400922450185 5.6464283762735334 0.8638038636710728 -> xyz=0.9665428940687371 0.9896372884871573 0.8568418066111094 rpy=0.12511119359624798 5.869302657479386 3.7471401696628437
- joint 23_to_11: axis 1 0 0 -> 0 1 0; origin xyz=0.6468384730736209 0.3982034764994321 0.6535115948109418 rpy=9.906013836752773 5.6464283762735334 0.8638038636710728 -> xyz=0.9665428940687371 0.9896372884871573 0.8568418066111094 rpy=0.18766679039437195 5.869302657479386 3.7471401696628437

File: temp2.urdf (robot description, URDF)
Before this commit: robot pepe, 1 links, 0 joints
Links:
- link 0: mass 0.32333990492988784 -> 0.19742596388519396; geometry collision cylinder length=0.9853454403519184 radius=0.2525416080782076; visual cylinder length=0.9853454403519184 radius=0.2525416080782076

File: temp3.urdf (robot description, URDF)
Before this commit: robot pepe, 4 links, 3 joints
Links:
- removed link 12
- removed link 13
- added link 18, mass 4.467304882838585e-06; collision cylinder length=1.9168577574955858 radius=0.0008612969648227331; visual cylinder length=1.9168577574955858 radius=0.0008612969648227331
- added link 212, mass 0.06126167348981085; collision cylinder length=1.9168577574955858 radius=0.10086129696482274; visual cylinder length=1.9168577574955858 radius=0.10086129696482274
- added link 22, mass 0.06126167348981085; collision cylinder length=1.9168577574955858 radius=0.10086129696482274; visual cylinder length=1.9168577574955858 radius=0.10086129696482274
- added link 25, mass 0.06126167348981085; collision cylinder length=1.9168577574955858 radius=0.10086129696482274; visual cylinder length=1.9168577574955858 radius=0.10086129696482274
- added link 29, mass 0.06126167348981085; collision cylinder length=1.9168577574955858 radius=0.10086129696482274; visual cylinder length=1.9168577574955858 radius=0.10086129696482274
- added link 310, mass 0.7177927362512388; collision cylinder length=0.40488831582507845 radius=0.7512024075422402; visual cylinder length=0.40488831582507845 radius=0.7512024075422402
- added link 311, mass 0.7177927362512388; collision cylinder length=0.40488831582507845 radius=0.7512024075422402; visual cylinder length=0.40488831582507845 radius=0.7512024075422402
- added link 313, mass 0.7177927362512388; collision cylinder length=0.40488831582507845 radius=0.7512024075422402; visual cylinder length=0.40488831582507845 radius=0.7512024075422402
- added link 314, mass 0.7177927362512388; collision cylinder length=0.40488831582507845 radius=0.7512024075422402; visual cylinder length=0.40488831582507845 radius=0.7512024075422402
- added link 33, mass 0.7177927362512388; collision cylinder length=0.40488831582507845 radius=0.7512024075422402; visual cylinder length=0.40488831582507845 radius=0.7512024075422402
- added link 34, mass 0.7177927362512388; collision cylinder length=0.40488831582507845 radius=0.7512024075422402; visual cylinder length=0.40488831582507845 radius=0.7512024075422402
- added link 36, mass 0.7177927362512388; collision cylinder length=0.40488831582507845 radius=0.7512024075422402; visual cylinder length=0.40488831582507845 radius=0.7512024075422402
- added link 37, mass 0.7177927362512388; collision cylinder length=0.40488831582507845 radius=0.7512024075422402; visual cylinder length=0.40488831582507845 radius=0.7512024075422402
- link 0: mass 1.038778327639143 -> 1.0360342360436707; geometry collision cylinder length=1.9998 radius=0.40608676477427597; visual cylinder length=1.9998 radius=0.40608676477427597
- link 11: mass 0.048116617275910635 -> 4.467304882838585e-06; geometry collision cylinder length=1.9168577574955858 radius=0.0008612969648227331; visual cylinder length=1.9168577574955858 radius=0.0008612969648227331
Joints:
- removed joint 12_to_0
- removed joint 13_to_0
- added joint 18_to_0: type revolute, parent 0, child 18, origin xyz=0.7236069504422373 0.9999 0.4161850445130292 rpy=5.3945979189771505 6.262356433276231 4.280533725595206, axis 0 1 0, limit lower=3.1415 upper=-3.1415 effort=1 velocity=1
- added joint 212_to_18: type revolute, parent 18, child 212, origin xyz=0.7236069504422373 0.9885880704038275 0.4161850445130292 rpy=7.2795535111310254 6.262356433276231 4.280533725595206, axis 0 1 0, limit lower=3.1415 upper=-3.1415 effort=1 velocity=1
- added joint 22_to_11: type revolute, parent 11, child 22, origin xyz=0.7236069504422373 0.9885880704038275 0.4161850445130292 rpy=4.853035674087351 6.262356433276231 4.280533725595206, axis 0 1 0, limit lower=3.1415 upper=-3.1415 effort=1 velocity=1
- added joint 25_to_11: type revolute, parent 11, child 25, origin xyz=0.7236069504422373 0.9885880704038275 0.4161850445130292 rpy=7.2795535111310254 6.262356433276231 4.280533725595206, axis 0 1 0, limit lower=3.1415 upper=-3.1415 effort=1 velocity=1
- added joint 29_to_18: type revolute, parent 18, child 29, origin xyz=0.7236069504422373 0.9885880704038275 0.4161850445130292 rpy=4.853035674087351 6.262356433276231 4.280533725595206, axis 0 1 0, limit lower=3.1415 upper=-3.1415 effort=1 velocity=1
- added joint 310_to_29: type revolute, parent 29, child 310, origin xyz=0.661355122961424 0.5316209256558981 0.2962522858232731 rpy=12.246047227773008 5.611737068211983 2.338051877508089, axis 0 1 0, limit lower=3.1415 upper=-3.1415 effort=1 velocity=1
- added joint 311_to_29: type revolute, parent 29, child 311, origin xyz=0.661355122961424 0.5316209256558981 0.2962522858232731 rpy=18.369070841659514 5.611737068211983 2.338051877508089, axis 0 1 0, limit lower=3.1415 upper=-3.1415 effort=1 velocity=1
- added joint 313_to_212: type revolute, parent 212, child 313, origin xyz=0.661355122961424 0.5316209256558981 0.2962522858232731 rpy=12.246047227773008 5.611737068211983 2.338051877508089, axis 0 1 0, limit lower=3.1415 upper=-3.1415 effort=1 velocity=1
- added joint 314_to_212: type revolute, parent 212, child 314, origin xyz=0.661355122961424 0.5316209256558981 0.2962522858232731 rpy=18.369070841659514 5.611737068211983 2.338051877508089, axis 0 1 0, limit lower=3.1415 upper=-3.1415 effort=1 velocity=1
- added joint 33_to_22: type revolute, parent 22, child 33, origin xyz=0.661355122961424 0.5316209256558981 0.2962522858232731 rpy=12.246047227773008 5.611737068211983 2.338051877508089, axis 0 1 0, limit lower=3.1415 upper=-3.1415 effort=1 velocity=1
- added joint 34_to_22: type revolute, parent 22, child 34, origin xyz=0.661355122961424 0.5316209256558981 0.2962522858232731 rpy=18.369070841659514 5.611737068211983 2.338051877508089, axis 0 1 0, limit lower=3.1415 upper=-3.1415 effort=1 velocity=1
- added joint 36_to_25: type revolute, parent 25, child 36, origin xyz=0.661355122961424 0.5316209256558981 0.2962522858232731 rpy=12.246047227773008 5.611737068211983 2.338051877508089, axis 0 1 0, limit lower=3.1415 upper=-3.1415 effort=1 velocity=1
- added joint 37_to_25: type revolute, parent 25, child 37, origin xyz=0.661355122961424 0.5316209256558981 0.2962522858232731 rpy=18.369070841659514 5.611737068211983 2.338051877508089, axis 0 1 0, limit lower=3.1415 upper=-3.1415 effort=1 velocity=1
- joint 11_to_0: axis 0 0 1 -> 0 1 0; origin xyz=0.5346921704194656 0.7675536365303309 0.03727917973075667 rpy=5.6612653984215715 3.1699043910322446 0.44175665736072767 -> xyz=0.7236069504422373 0.9999 0.4161850445130292 rpy=3.596398612651434 6.262356433276231 4.280533725595206

File: temp4.urdf (robot description, URDF)
Before this commit: robot pepe, 1 links, 0 joints
Links:
- added link 11, mass 0.3066418042690306; collision cylinder length=0.7853454403519184 radius=0.35254160807820756; visual cylinder length=0.7853454403519184 radius=0.35254160807820756
- link 0: mass 0.2886000077562378 -> 1.0360342360436707; geometry collision cylinder length=1.9998 radius=0.40608676477427597; visual cylinder length=1.9998 radius=0.40608676477427597
Joints:
- added joint 11_to_0: type revolute, parent 0, child 11, origin xyz=0.43638400265132093 0.035632360108815986 0.31232581489814226 rpy=11.059927898506901 2.536670462446014 1.6217615205138476, axis 0 0 1, limit lower=3.1415 upper=-3.1415 effort=1 velocity=1

File: temp5.urdf (robot description, URDF)
Before this commit: robot pepe, 7 links, 6 joints
Links:
- removed link 11
- removed link 12
- removed link 13
- removed link 24
- removed link 25
- removed link 26
- link 0: mass 3.012449546198092 -> 0.19742596388519396; geometry collision cylinder length=0.9853454403519184 radius=0.2525416080782076; visual cylinder length=0.9853454403519184 radius=0.2525416080782076
Joints:
- removed joint 11_to_0
- removed joint 12_to_0
- removed joint 13_to_0
- removed joint 24_to_0
- removed joint 25_to_0
- removed joint 26_to_0

File: temp6.urdf (robot description, URDF)
Before this commit: robot pepe, 1 links, 0 joints
Links:
- added link 11, mass 0.3066418042690306; collision cylinder length=0.7853454403519184 radius=0.35254160807820756; visual cylinder length=0.7853454403519184 radius=0.35254160807820756
- link 0: mass 0.32333990492988784 -> 0.5560741273262054; geometry collision cylinder length=1.2481208226524536 radius=0.3765850662787882; visual cylinder length=1.2481208226524536 radius=0.3765850662787882
Joints:
- added joint 11_to_0: type revolute, parent 0, child 11, origin xyz=0.33638400265132096 0.035632360108815986 0.41232581489814224 rpy=12.316564959942818 2.536670462446014 2.250080051231806, axis 0 0 1, limit lower=3.1415 upper=-3.1415 effort=1 velocity=1

File: temp7.urdf (robot description, URDF)
Before this commit: robot pepe, 13 links, 12 joints
Links:
- removed link 15
- removed link 19
- removed link 210
- removed link 211
- removed link 212
- removed link 24
- removed link 26
- removed link 27
- removed link 28
- link 0: mass 3.012449546198092 -> 0.018782858160138177; geometry collision cylinder length=0.547019036610694 radius=0.10454534086455025; visual cylinder length=0.547019036610694 radius=0.10454534086455025
- link 11: mass 0.32333990492988784 -> 0.15735352719442636; geometry collision cylinder length=0.7853454403519184 radius=0.2525416080782076; visual cylinder length=0.7853454403519184 radius=0.2525416080782076
- link 22: mass 0.605610648863151 -> 0.6435100811794822; geometry collision cylinder length=0.4221688028635415 radius=0.6965618303238383; visual cylinder length=0.4221688028635415 radius=0.6965618303238383
- link 23: mass 0.605610648863151 -> 0.6435100811794822; geometry collision cylinder length=0.4221688028635415 radius=0.6965618303238383; visual cylinder length=0.4221688028635415 radius=0.6965618303238383
Joints:
- removed joint 15_to_0
- removed joint 19_to_0
- removed joint 210_to_19
- removed joint 211_to_19
- removed joint 212_to_19
- removed joint 22_to_11
- removed joint 23_to_11
- removed joint 24_to_11
- removed joint 26_to_15
- removed joint 27_to_15
- removed joint 28_to_15
- added joint 22_to_0: type revolute, parent 0, child 22, origin xyz=0.7023675420825124 0.31866726646145793 0.49911583947315474 rpy=16.402647014181913 4.34539645277712 3.739331143605401, axis 0 0 1, limit lower=3.1415 upper=-3.1415 effort=1 velocity=1
- added joint 23_to_0: type revolute, parent 0, child 23, origin xyz=0.7023675420825124 0.31866726646145793 0.49911583947315474 rpy=21.870196018909215 4.34539645277712 3.739331143605401, axis 0 0 1, limit lower=3.1415 upper=-3.1415 effort=1 velocity=1
- joint 11_to_0: axis 1 0 0 -> 0 0 1; origin xyz=0.6468384730736209 0.3982034764994321 0.6535115948109418 rpy=5.347372163065932 5.018109845555575 0.8638038636710728 -> xyz=0.33638400265132096 0.035632360108815986 0.31232581489814226 rpy=11.059927898506901 2.536670462446014 2.250080051231806
