Commit message: reduce experiments

File: temp5.urdf (robot description, URDF)
Before this commit: robot pepe, 13 links, 12 joints
Links:
- link 0: mass 0.0637264246388024 -> 0.0006625578457586183; geometry collision cylinder length=1.9998 radius=0.010269367177534572; visual cylinder length=1.9998 radius=0.010269367177534572
- link 210: mass 6.281300540076709 -> 2.9750240410745246; geometry collision cylinder length=1.9005037910659992 radius=0.7058882183069434; visual cylinder length=1.9005037910659992 radius=0.7058882183069434
- link 211: mass 6.281300540076709 -> 2.9750240410745246; geometry collision cylinder length=1.9005037910659992 radius=0.7058882183069434; visual cylinder length=1.9005037910659992 radius=0.7058882183069434
- link 212: mass 6.281300540076709 -> 2.9750240410745246; geometry collision cylinder length=1.9005037910659992 radius=0.7058882183069434; visual cylinder length=1.9005037910659992 radius=0.7058882183069434
- link 22: mass 6.281300540076709 -> 2.9750240410745246; geometry collision cylinder length=1.9005037910659992 radius=0.7058882183069434; visual cylinder length=1.9005037910659992 radius=0.7058882183069434
- link 23: mass 6.281300540076709 -> 2.9750240410745246; geometry collision cylinder length=1.9005037910659992 radius=0.7058882183069434; visual cylinder length=1.9005037910659992 radius=0.7058882183069434
- link 24: mass 6.281300540076709 -> 2.9750240410745246; geometry collision cylinder length=1.9005037910659992 radius=0.7058882183069434; visual cylinder length=1.9005037910659992 radius=0.7058882183069434
- link 26: mass 6.281300540076709 -> 2.9750240410745246; geometry collision cylinder length=1.9005037910659992 radius=0.7058882183069434; visual cylinder length=1.9005037910659992 radius=0.7058882183069434
- link 27: mass 6.281300540076709 -> 2.9750240410745246; geometry collision cylinder length=1.9005037910659992 radius=0.7058882183069434; visual cylinder length=1.9005037910659992 radius=0.7058882183069434
- link 28: mass 6.281300540076709 -> 2.9750240410745246; geometry collision cylinder length=1.9005037910659992 radius=0.7058882183069434; visual cylinder length=1.9005037910659992 radius=0.7058882183069434
Joints:
- joint 11_to_0: axis 0 0 1 -> 1 0 0; origin xyz=0.9999 0.9999 0.9999 rpy=12.565113977297736 6.282556988648868 6.282556988648868 -> xyz=0.6849810317268884 0.4262293513728075 0.9999 rpy=10.00547663531266 4.364559318388451 3.6585971237677777
- joint 15_to_0: axis 0 0 1 -> 1 0 0; origin xyz=0.9999 0.9999 0.9999 rpy=18.847670965946605 6.282556988648868 6.282556988648868 -> xyz=0.6849810317268884 0.4262293513728075 0.9999 rpy=15.008214952968988 4.364559318388451 3.6585971237677777
- joint 19_to_0: axis 0 0 1 -> 1 0 0; origin xyz=0.9999 0.9999 0.9999 rpy=25.130227954595473 6.282556988648868 6.282556988648868 -> xyz=0.6849810317268884 0.4262293513728075 0.9999 rpy=20.01095327062532 4.364559318388451 3.6585971237677777
- joint 210_to_19: axis 0 0 1 -> 1 0 0; origin xyz=0.9999 0.9999 0.9999 rpy=12.565113977297736 6.282556988648868 6.282556988648868 -> xyz=0.2506740408016117 0.09067578195260384 0.9286167875098919 rpy=1.74701695915431 4.495996032334981 5.787035230481515
- joint 211_to_19: axis 0 0 1 -> 1 0 0; origin xyz=0.9999 0.9999 0.9999 rpy=18.847670965946605 6.282556988648868 6.282556988648868 -> xyz=0.2506740408016117 0.09067578195260384 0.9286167875098919 rpy=2.620525438731465 4.495996032334981 5.787035230481515
- joint 212_to_19: axis 0 0 1 -> 1 0 0; origin xyz=0.9999 0.9999 0.9999 rpy=25.130227954595473 6.282556988648868 6.282556988648868 -> xyz=0.2506740408016117 0.09067578195260384 0.9286167875098919 rpy=3.49403391830862 4.495996032334981 5.787035230481515
- joint 22_to_11: axis 0 0 1 -> 1 0 0; origin xyz=0.9999 0.9999 0.9999 rpy=12.565113977297736 6.282556988648868 6.282556988648868 -> xyz=0.2506740408016117 0.09067578195260384 0.9286167875098919 rpy=1.74701695915431 4.495996032334981 5.787035230481515
- joint 23_to_11: axis 0 0 1 -> 1 0 0; origin xyz=0.9999 0.9999 0.9999 rpy=18.847670965946605 6.282556988648868 6.282556988648868 -> xyz=0.2506740408016117 0.09067578195260384 0.9286167875098919 rpy=2.620525438731465 4.495996032334981 5.787035230481515
- joint 24_to_11: axis 0 0 1 -> 1 0 0; origin xyz=0.9999 0.9999 0.9999 rpy=25.130227954595473 6.282556988648868 6.282556988648868 -> xyz=0.2506740408016117 0.09067578195260384 0.9286167875098919 rpy=3.49403391830862 4.495996032334981 5.787035230481515
- joint 26_to_15: axis 0 0 1 -> 1 0 0; origin xyz=0.9999 0.9999 0.9999 rpy=12.565113977297736 6.282556988648868 6.282556988648868 -> xyz=0.2506740408016117 0.09067578195260384 0.9286167875098919 rpy=1.74701695915431 4.495996032334981 5.787035230481515
- joint 27_to_15: axis 0 0 1 -> 1 0 0; origin xyz=0.9999 0.9999 0.9999 rpy=18.847670965946605 6.282556988648868 6.282556988648868 -> xyz=0.2506740408016117 0.09067578195260384 0.9286167875098919 rpy=2.620525438731465 4.495996032334981 5.787035230481515
- joint 28_to_15: axis 0 0 1 -> 1 0 0; origin xyz=0.9999 0.9999 0.9999 rpy=25.130227954595473 6.282556988648868 6.282556988648868 -> xyz=0.2506740408016117 0.09067578195260384 0.9286167875098919 rpy=3.49403391830862 4.495996032334981 5.787035230481515

File: temp6.urdf (robot description, URDF)
Before this commit: robot pepe, 13 links, 12 joints
Links:
- removed link 15
- removed link 19
- removed link 210
- removed link 211
- removed link 212
- removed link 22
- removed link 23
- removed link 24
- removed link 26
- removed link 27
- removed link 28
- added link 12, mass 6.281300540076709; collision cylinder length=1.9998 radius=0.9999; visual cylinder length=1.9998 radius=0.9999
- added link 13, mass 6.281300540076709; collision cylinder length=1.9998 radius=0.9999; visual cylinder length=1.9998 radius=0.9999
- link 0: mass 0.00019415638996012175 -> 0.4092927598651034; geometry collision cylinder length=0.46564214033996487 radius=0.5289516258890312; visual cylinder length=0.46564214033996487 radius=0.5289516258890312
- link 11: mass 0.0637264246388024 -> 6.281300540076709; geometry collision cylinder length=1.9998 radius=0.9999; visual cylinder length=1.9998 radius=0.9999
Joints:
- removed joint 15_to_0
- removed joint 19_to_0
- removed joint 210_to_19
- removed joint 211_to_19
- removed joint 212_to_19
- removed joint 22_to_11
- removed joint 23_to_11
- removed joint 24_to_11
- removed joint 26_to_15
- removed joint 27_to_15
- removed joint 28_to_15
- added joint 12_to_0: type revolute, parent 0, child 12, origin xyz=0.6849810317268884 0.32622935137280745 0.9999 rpy=15.008214952968988 4.364559318388451 3.6585971237677777, axis 1 0 0, limit lower=3.1415 upper=-3.1415 effort=1 velocity=1
- added joint 13_to_0: type revolute, parent 0, child 13, origin xyz=0.6849810317268884 0.32622935137280745 0.9999 rpy=20.01095327062532 4.364559318388451 3.6585971237677777, axis 1 0 0, limit lower=3.1415 upper=-3.1415 effort=1 velocity=1
- joint 11_to_0: axis 0 0 1 -> 1 0 0; origin xyz=0.8963054758440083 0.9999 0.9999 rpy=12.565113977297736 6.282556988648868 6.282556988648868 -> xyz=0.6849810317268884 0.32622935137280745 0.9999 rpy=10.00547663531266 4.364559318388451 3.6585971237677777

File: temp7.urdf (robot description, URDF)
Before this commit: robot pepe, 1 links, 0 joints
Links:
- added link 11, mass 0.0006625578457586183; collision cylinder length=1.9998 radius=0.010269367177534572; visual cylinder length=1.9998 radius=0.010269367177534572
- added link 15, mass 0.0006625578457586183; collision cylinder length=1.9998 radius=0.010269367177534572; visual cylinder length=1.9998 radius=0.010269367177534572
- added link 22, mass 6.281300540076709; collision cylinder length=1.9998 radius=0.9999; visual cylinder length=1.9998 radius=0.9999
- added link 23, mass 6.281300540076709; collision cylinder length=1.9998 radius=0.9999; visual cylinder length=1.9998 radius=0.9999
- added link 24, mass 6.281300540076709; collision cylinder length=1.9998 radius=0.9999; visual cylinder length=1.9998 radius=0.9999
- added link 26, mass 6.281300540076709; collision cylinder length=1.9998 radius=0.9999; visual cylinder length=1.9998 radius=0.9999
- added link 27, mass 6.281300540076709; collision cylinder length=1.9998 radius=0.9999; visual cylinder length=1.9998 radius=0.9999
- added link 28, mass 6.281300540076709; collision cylinder length=1.9998 radius=0.9999; visual cylinder length=1.9998 radius=0.9999
- link 0: mass 6.281300540076709 -> 1.5531439629661394; geometry collision cylinder length=0.6649032241420763 radius=0.8622867260735491; visual cylinder length=0.6649032241420763 radius=0.8622867260735491
Joints:
- added joint 11_to_0: type revolute, parent 0, child 11, origin xyz=0.819504762628304 0.48519491423040395 0.9999 rpy=8.735078713834518 3.5719656927887087 6.147482522451077, axis 0 0 1, limit lower=3.1415 upper=-3.1415 effort=1 velocity=1
- added joint 15_to_0: type revolute, parent 0, child 15, origin xyz=0.819504762628304 0.48519491423040395 0.9999 rpy=13.102618070751777 3.5719656927887087 6.147482522451077, axis 0 0 1, limit lower=3.1415 upper=-3.1415 effort=1 velocity=1
- added joint 22_to_11: type revolute, parent 11, child 22, origin xyz=0.6849810317268884 0.32622935137280745 0.9999 rpy=10.00547663531266 4.992877849106409 3.6585971237677777, axis 1 0 0, limit lower=3.1415 upper=-3.1415 effort=1 velocity=1
- added joint 23_to_11: type revolute, parent 11, child 23, origin xyz=0.6849810317268884 0.32622935137280745 0.9999 rpy=15.008214952968988 4.992877849106409 3.6585971237677777, axis 1 0 0, limit lower=3.1415 upper=-3.1415 effort=1 velocity=1
- added joint 24_to_11: type revolute, parent 11, child 24, origin xyz=0.6849810317268884 0.32622935137280745 0.9999 rpy=20.01095327062532 4.992877849106409 3.6585971237677777, axis 1 0 0, limit lower=3.1415 upper=-3.1415 effort=1 velocity=1
- added joint 26_to_15: type revolute, parent 15, child 26, origin xyz=0.6849810317268884 0.32622935137280745 0.9999 rpy=10.00547663531266 4.992877849106409 3.6585971237677777, axis 1 0 0, limit lower=3.1415 upper=-3.1415 effort=1 velocity=1
- added joint 27_to_15: type revolute, parent 15, child 27, origin xyz=0.6849810317268884 0.32622935137280745 0.9999 rpy=15.008214952968988 4.992877849106409 3.6585971237677777, axis 1 0 0, limit lower=3.1415 upper=-3.1415 effort=1 velocity=1
- added joint 28_to_15: type revolute, parent 15, child 28, origin xyz=0.6849810317268884 0.32622935137280745 0.9999 rpy=20.01095327062532 4.992877849106409 3.6585971237677777, axis 1 0 0, limit lower=3.1415 upper=-3.1415 effort=1 velocity=1

File: temp9.urdf (robot description, URDF)
Before this commit: robot pepe, 13 links, 12 joints
Links:
- link 0: mass 6.281300540076709 -> 0.00019415638996012175; geometry collision cylinder length=0.20469765564289283 radius=0.01737578657019445; visual cylinder length=0.20469765564289283 radius=0.01737578657019445
