Commit message: save intermediate results

File: temp0.urdf (robot description, URDF)
Before this commit: robot pepe, 37 links, 36 joints
Links:
- removed link 1017
- removed link 1022
- removed link 1027
- removed link 1134
- removed link 15
- removed link 19
- removed link 213
- removed link 218
- removed link 223
- removed link 328
- removed link 330
- removed link 410
- removed link 411
- removed link 412
- removed link 42
- removed link 43
- removed link 44
- removed link 46
- removed link 47
- removed link 48
- removed link 532
- removed link 614
- removed link 615
- removed link 616
- removed link 619
- removed link 620
- removed link 621
- removed link 624
- removed link 625
- removed link 626
- removed link 735
- removed link 736
- removed link 833
- removed link 929
- removed link 931
- link 0: mass 0.7173020552644698 -> 0.1266493789566258; geometry collision cylinder length=1.2050055825401313 radius=0.18290773275572914; visual cylinder length=1.2050055825401313 radius=0.18290773275572914
- link 11: mass 3.1339990824625334 -> 2.561384175740279; geometry collision cylinder length=0.8154769926966201 radius=0.9999; visual cylinder length=0.8154769926966201 radius=0.9999
Joints:
- removed joint 1017_to_213
- removed joint 1022_to_218
- removed joint 1027_to_223
- removed joint 1134_to_833
- removed joint 15_to_0
- removed joint 19_to_0
- removed joint 213_to_0
- removed joint 218_to_0
- removed joint 223_to_0
- removed joint 328_to_0
- removed joint 330_to_0
- removed joint 410_to_19
- removed joint 411_to_19
- removed joint 412_to_19
- removed joint 42_to_11
- removed joint 43_to_11
- removed joint 44_to_11
- removed joint 46_to_15
- removed joint 47_to_15
- removed joint 48_to_15
- removed joint 532_to_0
- removed joint 614_to_213
- removed joint 615_to_213
- removed joint 616_to_213
- removed joint 619_to_218
- removed joint 620_to_218
- removed joint 621_to_218
- removed joint 624_to_223
- removed joint 625_to_223
- removed joint 626_to_223
- removed joint 735_to_0
- removed joint 736_to_0
- removed joint 833_to_532
- removed joint 929_to_328
- removed joint 931_to_330
- joint 11_to_0: axis 1 0 0 -> 0 1 0; origin xyz=0.68566985513273 0.5064215327422712 0.4388266654996933 rpy=9.032049515710266 2.55451078082068 3.1761236737343506 -> xyz=0.5488228574833086 0.7727352694338915 0.9999 rpy=9.187154749586885 4.526911794548183 5.196853465412705

File: temp1.urdf (robot description, URDF)
Before this commit: robot pepe, 82 links, 81 joints
Links:
- removed link 1032
- removed link 1033
- removed link 1053
- removed link 1054
- removed link 1074
- removed link 1075
- removed link 1177
- removed link 1178
- removed link 1180
- removed link 1181
- removed link 15
- removed link 19
- removed link 213
- removed link 234
- removed link 255
- removed link 376
- removed link 379
- removed link 414
- removed link 422
- removed link 435
- removed link 443
- removed link 456
- removed link 464
- removed link 515
- removed link 518
- removed link 523
- removed link 526
- removed link 536
- removed link 539
- removed link 544
- removed link 547
- removed link 557
- removed link 560
- removed link 565
- removed link 568
- removed link 621
- removed link 629
- removed link 642
- removed link 650
- removed link 663
- removed link 671
- removed link 710
- removed link 711
- removed link 712
- removed link 72
- removed link 73
- removed link 74
- removed link 76
- removed link 77
- removed link 78
- removed link 816
- removed link 817
- removed link 819
- removed link 820
- removed link 824
- removed link 825
- removed link 827
- removed link 828
- removed link 837
- removed link 838
- removed link 840
- removed link 841
- removed link 845
- removed link 846
- removed link 848
- removed link 849
- removed link 858
- removed link 859
- removed link 861
- removed link 862
- removed link 866
- removed link 867
- removed link 869
- removed link 870
- removed link 930
- removed link 931
- removed link 951
- removed link 952
- removed link 972
- removed link 973
- added link 12, mass 0.1266493789566258; collision cylinder length=1.2050055825401313 radius=0.18290773275572914; visual cylinder length=1.2050055825401313 radius=0.18290773275572914
- added link 13, mass 0.1266493789566258; collision cylinder length=1.2050055825401313 radius=0.18290773275572914; visual cylinder length=1.2050055825401313 radius=0.18290773275572914
- link 0: mass 1.1291090016399166 -> 2.561384175740279; geometry collision cylinder length=0.8154769926966201 radius=0.9999; visual cylinder length=0.8154769926966201 radius=0.9999
- link 11: mass 0.37585443447588623 -> 0.1266493789566258; geometry collision cylinder length=1.2050055825401313 radius=0.18290773275572914; visual cylinder length=1.2050055825401313 radius=0.18290773275572914
Joints:
- removed joint 1032_to_213
- removed joint 1033_to_213
- removed joint 1053_to_234
- removed joint 1054_to_234
- removed joint 1074_to_255
- removed joint 1075_to_255
- removed joint 1177_to_376
- removed joint 1178_to_376
- removed joint 1180_to_379
- removed joint 1181_to_379
- removed joint 15_to_0
- removed joint 19_to_0
- removed joint 213_to_0
- removed joint 234_to_0
- removed joint 255_to_0
- removed joint 376_to_0
- removed joint 379_to_0
- removed joint 414_to_213
- removed joint 422_to_213
- removed joint 435_to_234
- removed joint 443_to_234
- removed joint 456_to_255
- removed joint 464_to_255
- removed joint 515_to_414
- removed joint 518_to_414
- removed joint 523_to_422
- removed joint 526_to_422
- removed joint 536_to_435
- removed joint 539_to_435
- removed joint 544_to_443
- removed joint 547_to_443
- removed joint 557_to_456
- removed joint 560_to_456
- removed joint 565_to_464
- removed joint 568_to_464
- removed joint 621_to_414
- removed joint 629_to_422
- removed joint 642_to_435
- removed joint 650_to_443
- removed joint 663_to_456
- removed joint 671_to_464
- removed joint 710_to_19
- removed joint 711_to_19
- removed joint 712_to_19
- removed joint 72_to_11
- removed joint 73_to_11
- removed joint 74_to_11
- removed joint 76_to_15
- removed joint 77_to_15
- removed joint 78_to_15
- removed joint 816_to_515
- removed joint 817_to_515
- removed joint 819_to_518
- removed joint 820_to_518
- removed joint 824_to_523
- removed joint 825_to_523
- removed joint 827_to_526
- removed joint 828_to_526
- removed joint 837_to_536
- removed joint 838_to_536
- removed joint 840_to_539
- removed joint 841_to_539
- removed joint 845_to_544
- removed joint 846_to_544
- removed joint 848_to_547
- removed joint 849_to_547
- removed joint 858_to_557
- removed joint 859_to_557
- removed joint 861_to_560
- removed joint 862_to_560
- removed joint 866_to_565
- removed joint 867_to_565
- removed joint 869_to_568
- removed joint 870_to_568
- removed joint 930_to_213
- removed joint 931_to_213
- removed joint 951_to_234
- removed joint 952_to_234
- removed joint 972_to_255
- removed joint 973_to_255
- added joint 12_to_0: type revolute, parent 0, child 12, origin xyz=0.29548778666124453 0.12065575549339036 0.5154713031273903 rpy=7.375138112199213 4.924491704359826 3.0762963088839346, axis 0 1 0, limit lower=3.1415 upper=-3.1415 effort=1 velocity=1
- added joint 13_to_0: type revolute, parent 0, child 13, origin xyz=0.29548778666124453 0.12065575549339036 0.5154713031273903 rpy=9.833517482932285 4.924491704359826 3.0762963088839346, axis 0 1 0, limit lower=3.1415 upper=-3.1415 effort=1 velocity=1
- joint 11_to_0: origin xyz=0.23435510414376926 0.022349168043231726 0.040616981490420034 rpy=1.3516872645789864 1.6363588624652674 1.7721646499765726 -> xyz=0.29548778666124453 0.12065575549339036 0.5154713031273903 rpy=4.9167587414661424 4.924491704359826 3.0762963088839346

File: temp2.urdf (robot description, URDF)
Before this commit: robot pepe, 143 links, 142 joints
Links:
- removed link 1010
- removed link 1011
- removed link 1019
- removed link 1020
- removed link 1021
- removed link 109
- removed link 11
- removed link 11100
- removed link 11101
- removed link 11102
- removed link 11106
- removed link 11107
- removed link 11108
- removed link 11110
- removed link 11111
- removed link 11112
- removed link 11114
- removed link 11115
- removed link 11116
- removed link 11119
- removed link 11120
- removed link 11121
- removed link 11123
- removed link 11124
- removed link 11125
- removed link 11127
- removed link 11128
- removed link 11129
- removed link 11132
- removed link 11133
- removed link 11134
- removed link 11136
- removed link 11137
- removed link 11138
- removed link 11140
- removed link 11141
- removed link 11142
- removed link 1126
- removed link 1127
- removed link 1128
- removed link 1130
- removed link 1131
- removed link 1132
- removed link 1134
- removed link 1135
- removed link 1136
- removed link 1139
- removed link 1140
- removed link 1141
- removed link 1143
- removed link 1144
- removed link 1145
- removed link 1147
- removed link 1148
- removed link 1149
- removed link 1152
- removed link 1153
- removed link 1154
- removed link 1156
- removed link 1157
- removed link 1158
- removed link 1160
- removed link 1161
- removed link 1162
- removed link 1166
- removed link 1167
- removed link 1168
- removed link 1170
- removed link 1171
- removed link 1172
- removed link 1174
- removed link 1175
- removed link 1176
- removed link 1179
- removed link 1180
- removed link 1181
- removed link 1183
- removed link 1184
- removed link 1185
- removed link 1187
- removed link 1188
- removed link 1189
- removed link 1192
- removed link 1193
- removed link 1194
- removed link 1196
- removed link 1197
- removed link 1198
- removed link 212
- removed link 22
- removed link 313
- removed link 314
- removed link 315
- removed link 33
- removed link 34
- removed link 35
- removed link 416
- removed link 417
- removed link 46
- removed link 47
- removed link 522
- removed link 6103
- removed link 623
- removed link 663
- removed link 718
- removed link 78
- removed link 8104
- removed link 8117
- removed link 8130
- removed link 824
- removed link 837
- removed link 850
- removed link 864
- removed link 877
- removed link 890
- removed link 9105
- removed link 9109
- removed link 9113
- removed link 9118
- removed link 9122
- removed link 9126
- removed link 9131
- removed link 9135
- removed link 9139
- removed link 925
- removed link 929
- removed link 933
- removed link 938
- removed link 942
- removed link 946
- removed link 951
- removed link 955
- removed link 959
- removed link 965
- removed link 969
- removed link 973
- removed link 978
- removed link 982
- removed link 986
- removed link 991
- removed link 995
- removed link 999
- link 0: mass 0.051061698887551785 -> 2.6568424106949546; geometry collision cylinder length=1.01547699269662 radius=0.9125841407500055; visual cylinder length=1.01547699269662 radius=0.9125841407500055
Joints:
- removed joint 1010_to_78
- removed joint 1011_to_78
- removed joint 1019_to_718
- removed joint 1020_to_718
- removed joint 1021_to_718
- removed joint 109_to_78
- removed joint 11100_to_999
- removed joint 11101_to_999
- removed joint 11102_to_999
- removed joint 11106_to_9105
- removed joint 11107_to_9105
- removed joint 11108_to_9105
- removed joint 11110_to_9109
- removed joint 11111_to_9109
- removed joint 11112_to_9109
- removed joint 11114_to_9113
- removed joint 11115_to_9113
- removed joint 11116_to_9113
- removed joint 11119_to_9118
- removed joint 11120_to_9118
- removed joint 11121_to_9118
- removed joint 11123_to_9122
- removed joint 11124_to_9122
- removed joint 11125_to_9122
- removed joint 11127_to_9126
- removed joint 11128_to_9126
- removed joint 11129_to_9126
- removed joint 11132_to_9131
- removed joint 11133_to_9131
- removed joint 11134_to_9131
- removed joint 11136_to_9135
- removed joint 11137_to_9135
- removed joint 11138_to_9135
- removed joint 11140_to_9139
- removed joint 11141_to_9139
- removed joint 11142_to_9139
- removed joint 1126_to_925
- removed joint 1127_to_925
- removed joint 1128_to_925
- removed joint 1130_to_929
- removed joint 1131_to_929
- removed joint 1132_to_929
- removed joint 1134_to_933
- removed joint 1135_to_933
- removed joint 1136_to_933
- removed joint 1139_to_938
- removed joint 1140_to_938
- removed joint 1141_to_938
- removed joint 1143_to_942
- removed joint 1144_to_942
- removed joint 1145_to_942
- removed joint 1147_to_946
- removed joint 1148_to_946
- removed joint 1149_to_946
- removed joint 1152_to_951
- removed joint 1153_to_951
- removed joint 1154_to_951
- removed joint 1156_to_955
- removed joint 1157_to_955
- removed joint 1158_to_955
- removed joint 1160_to_959
- removed joint 1161_to_959
- removed joint 1162_to_959
- removed joint 1166_to_965
- removed joint 1167_to_965
- removed joint 1168_to_965
- removed joint 1170_to_969
- removed joint 1171_to_969
- removed joint 1172_to_969
- removed joint 1174_to_973
- removed joint 1175_to_973
- removed joint 1176_to_973
- removed joint 1179_to_978
- removed joint 1180_to_978
- removed joint 1181_to_978
- removed joint 1183_to_982
- removed joint 1184_to_982
- removed joint 1185_to_982
- removed joint 1187_to_986
- removed joint 1188_to_986
- removed joint 1189_to_986
- removed joint 1192_to_991
- removed joint 1193_to_991
- removed joint 1194_to_991
- removed joint 1196_to_995
- removed joint 1197_to_995
- removed joint 1198_to_995
- removed joint 11_to_0
- removed joint 212_to_0
- removed joint 22_to_0
- removed joint 313_to_212
- removed joint 314_to_212
- removed joint 315_to_212
- removed joint 33_to_22
- removed joint 34_to_22
- removed joint 35_to_22
- removed joint 416_to_212
- removed joint 417_to_212
- removed joint 46_to_22
- removed joint 47_to_22
- removed joint 522_to_0
- removed joint 6103_to_522
- removed joint 623_to_522
- removed joint 663_to_522
- removed joint 718_to_212
- removed joint 78_to_22
- removed joint 8104_to_6103
- removed joint 8117_to_6103
- removed joint 8130_to_6103
- removed joint 824_to_623
- removed joint 837_to_623
- removed joint 850_to_623
- removed joint 864_to_663
- removed joint 877_to_663
- removed joint 890_to_663
- removed joint 9105_to_8104
- removed joint 9109_to_8104
- removed joint 9113_to_8104
- removed joint 9118_to_8117
- removed joint 9122_to_8117
- removed joint 9126_to_8117
- removed joint 9131_to_8130
- removed joint 9135_to_8130
- removed joint 9139_to_8130
- removed joint 925_to_824
- removed joint 929_to_824
- removed joint 933_to_824
- removed joint 938_to_837
- removed joint 942_to_837
- removed joint 946_to_837
- removed joint 951_to_850
- removed joint 955_to_850
- removed joint 959_to_850
- removed joint 965_to_864
- removed joint 969_to_864
- removed joint 973_to_864
- removed joint 978_to_877
- removed joint 982_to_877
- removed joint 986_to_877
- removed joint 991_to_890
- removed joint 995_to_890
- removed joint 999_to_890

File: temp3.urdf (robot description, URDF)
Before this commit: robot pepe, 79 links, 78 joints
Links:
- removed link 1012
- removed link 1013
- removed link 1014
- removed link 1018
- removed link 1019
- removed link 1020
- removed link 1045
- removed link 1046
- removed link 1047
- removed link 1051
- removed link 1052
- removed link 1053
- removed link 1057
- removed link 1058
- removed link 1059
- removed link 106
- removed link 107
- removed link 108
- removed link 11
- removed link 1137
- removed link 1138
- removed link 1139
- removed link 1176
- removed link 1177
- removed link 1178
- removed link 140
- removed link 22
- removed link 241
- removed link 327
- removed link 331
- removed link 366
- removed link 370
- removed link 415
- removed link 43
- removed link 442
- removed link 448
- removed link 454
- removed link 49
- removed link 535
- removed link 536
- removed link 574
- removed link 575
- removed link 621
- removed link 623
- removed link 625
- removed link 660
- removed link 662
- removed link 664
- removed link 710
- removed link 711
- removed link 716
- removed link 717
- removed link 74
- removed link 743
- removed link 744
- removed link 749
- removed link 75
- removed link 750
- removed link 755
- removed link 756
- removed link 822
- removed link 824
- removed link 826
- removed link 861
- removed link 863
- removed link 865
- removed link 928
- removed link 929
- removed link 930
- removed link 932
- removed link 933
- removed link 934
- removed link 967
- removed link 968
- removed link 969
- removed link 971
- removed link 972
- removed link 973
- link 0: mass 0.23052126836723216 -> 2.561384175740279; geometry collision cylinder length=0.8154769926966201 radius=0.9999; visual cylinder length=0.8154769926966201 radius=0.9999
Joints:
- removed joint 1012_to_49
- removed joint 1013_to_49
- removed joint 1014_to_49
- removed joint 1018_to_415
- removed joint 1019_to_415
- removed joint 1020_to_415
- removed joint 1045_to_442
- removed joint 1046_to_442
- removed joint 1047_to_442
- removed joint 1051_to_448
- removed joint 1052_to_448
- removed joint 1053_to_448
- removed joint 1057_to_454
- removed joint 1058_to_454
- removed joint 1059_to_454
- removed joint 106_to_43
- removed joint 107_to_43
- removed joint 108_to_43
- removed joint 1137_to_11
- removed joint 1138_to_11
- removed joint 1139_to_11
- removed joint 1176_to_140
- removed joint 1177_to_140
- removed joint 1178_to_140
- removed joint 11_to_0
- removed joint 140_to_0
- removed joint 22_to_11
- removed joint 241_to_140
- removed joint 327_to_11
- removed joint 331_to_11
- removed joint 366_to_140
- removed joint 370_to_140
- removed joint 415_to_22
- removed joint 43_to_22
- removed joint 442_to_241
- removed joint 448_to_241
- removed joint 454_to_241
- removed joint 49_to_22
- removed joint 535_to_11
- removed joint 536_to_11
- removed joint 574_to_140
- removed joint 575_to_140
- removed joint 621_to_22
- removed joint 623_to_22
- removed joint 625_to_22
- removed joint 660_to_241
- removed joint 662_to_241
- removed joint 664_to_241
- removed joint 710_to_49
- removed joint 711_to_49
- removed joint 716_to_415
- removed joint 717_to_415
- removed joint 743_to_442
- removed joint 744_to_442
- removed joint 749_to_448
- removed joint 74_to_43
- removed joint 750_to_448
- removed joint 755_to_454
- removed joint 756_to_454
- removed joint 75_to_43
- removed joint 822_to_621
- removed joint 824_to_623
- removed joint 826_to_625
- removed joint 861_to_660
- removed joint 863_to_662
- removed joint 865_to_664
- removed joint 928_to_327
- removed joint 929_to_327
- removed joint 930_to_327
- removed joint 932_to_331
- removed joint 933_to_331
- removed joint 934_to_331
- removed joint 967_to_366
- removed joint 968_to_366
- removed joint 969_to_366
- removed joint 971_to_370
- removed joint 972_to_370
- removed joint 973_to_370

File: temp4.urdf (robot description, URDF)
Before this commit: robot pepe, 73 links, 72 joints
Links:
- removed link 1010
- removed link 1011
- removed link 1012
- removed link 1017
- removed link 1018
- removed link 1019
- removed link 1024
- removed link 1025
- removed link 1026
- removed link 1038
- removed link 1039
- removed link 1040
- removed link 1045
- removed link 1046
- removed link 1047
- removed link 1052
- removed link 1053
- removed link 1054
- removed link 1162
- removed link 1163
- removed link 1164
- removed link 1166
- removed link 1167
- removed link 1168
- removed link 1170
- removed link 1171
- removed link 1172
- removed link 13
- removed link 233
- removed link 25
- removed link 313
- removed link 320
- removed link 334
- removed link 341
- removed link 348
- removed link 36
- removed link 461
- removed link 465
- removed link 469
- removed link 514
- removed link 515
- removed link 516
- removed link 521
- removed link 522
- removed link 523
- removed link 535
- removed link 536
- removed link 537
- removed link 542
- removed link 543
- removed link 544
- removed link 549
- removed link 550
- removed link 551
- removed link 57
- removed link 58
- removed link 59
- removed link 627
- removed link 628
- removed link 655
- removed link 656
- removed link 729
- removed link 730
- removed link 757
- removed link 758
- removed link 831
- removed link 832
- removed link 859
- removed link 860
- removed link 92
- removed link 94
- link 0: mass 0.04137890269106453 -> 0.1266493789566258; geometry collision cylinder length=1.2050055825401313 radius=0.18290773275572914; visual cylinder length=1.2050055825401313 radius=0.18290773275572914
- link 11: mass 0.08663061389242722 -> 2.561384175740279; geometry collision cylinder length=0.8154769926966201 radius=0.9999; visual cylinder length=0.8154769926966201 radius=0.9999
Joints:
- removed joint 1010_to_36
- removed joint 1011_to_36
- removed joint 1012_to_36
- removed joint 1017_to_313
- removed joint 1018_to_313
- removed joint 1019_to_313
- removed joint 1024_to_320
- removed joint 1025_to_320
- removed joint 1026_to_320
- removed joint 1038_to_334
- removed joint 1039_to_334
- removed joint 1040_to_334
- removed joint 1045_to_341
- removed joint 1046_to_341
- removed joint 1047_to_341
- removed joint 1052_to_348
- removed joint 1053_to_348
- removed joint 1054_to_348
- removed joint 1162_to_461
- removed joint 1163_to_461
- removed joint 1164_to_461
- removed joint 1166_to_465
- removed joint 1167_to_465
- removed joint 1168_to_465
- removed joint 1170_to_469
- removed joint 1171_to_469
- removed joint 1172_to_469
- removed joint 13_to_0
- removed joint 233_to_0
- removed joint 25_to_0
- removed joint 313_to_25
- removed joint 320_to_25
- removed joint 334_to_233
- removed joint 341_to_233
- removed joint 348_to_233
- removed joint 36_to_25
- removed joint 461_to_0
- removed joint 465_to_0
- removed joint 469_to_0
- removed joint 514_to_313
- removed joint 515_to_313
- removed joint 516_to_313
- removed joint 521_to_320
- removed joint 522_to_320
- removed joint 523_to_320
- removed joint 535_to_334
- removed joint 536_to_334
- removed joint 537_to_334
- removed joint 542_to_341
- removed joint 543_to_341
- removed joint 544_to_341
- removed joint 549_to_348
- removed joint 550_to_348
- removed joint 551_to_348
- removed joint 57_to_36
- removed joint 58_to_36
- removed joint 59_to_36
- removed joint 627_to_25
- removed joint 628_to_25
- removed joint 655_to_233
- removed joint 656_to_233
- removed joint 729_to_25
- removed joint 730_to_25
- removed joint 757_to_233
- removed joint 758_to_233
- removed joint 831_to_25
- removed joint 832_to_25
- removed joint 859_to_233
- removed joint 860_to_233
- removed joint 92_to_11
- removed joint 94_to_13
- joint 11_to_0: axis 0 0 1 -> 0 1 0; origin xyz=0.43450033797431886 0.32400306826637915 0.7113008465722358 rpy=11.498078371534788 3.072462359084664 1.576784985733487 -> xyz=0.5488228574833086 0.6727352694338915 0.9037495979989713 rpy=9.187154749586885 4.526911794548183 5.196853465412705
