Commit message: save intermediate results

File: temp5.urdf (robot description, URDF)
Before this commit: robot pepe, 30 links, 29 joints
Links:
- removed link 1012
- removed link 1019
- removed link 105
- removed link 11
- removed link 1127
- removed link 1128
- removed link 1129
- removed link 115
- removed link 18
- removed link 216
- removed link 22
- removed link 29
- removed link 322
- removed link 323
- removed link 413
- removed link 414
- removed link 420
- removed link 421
- removed link 46
- removed link 47
- removed link 524
- removed link 610
- removed link 617
- removed link 63
- removed link 711
- removed link 718
- removed link 74
- removed link 825
- removed link 926
- link 0: mass 0.8598250831576532 -> 2.1335725720273833; geometry collision cylinder length=0.8154769926966201 radius=0.9125841407500055; visual cylinder length=0.8154769926966201 radius=0.9125841407500055
Joints:
- removed joint 1012_to_610
- removed joint 1019_to_617
- removed joint 105_to_63
- removed joint 1127_to_825
- removed joint 1128_to_825
- removed joint 1129_to_825
- removed joint 115_to_0
- removed joint 11_to_0
- removed joint 18_to_0
- removed joint 216_to_115
- removed joint 22_to_11
- removed joint 29_to_18
- removed joint 322_to_0
- removed joint 323_to_0
- removed joint 413_to_18
- removed joint 414_to_18
- removed joint 420_to_115
- removed joint 421_to_115
- removed joint 46_to_11
- removed joint 47_to_11
- removed joint 524_to_0
- removed joint 610_to_29
- removed joint 617_to_216
- removed joint 63_to_22
- removed joint 711_to_610
- removed joint 718_to_617
- removed joint 74_to_63
- removed joint 825_to_0
- removed joint 926_to_825

File: temp6.urdf (robot description, URDF)
Before this commit: robot pepe, 65 links, 64 joints
Links:
- removed link 1049
- removed link 1050
- removed link 1051
- removed link 1053
- removed link 1054
- removed link 1055
- removed link 11
- removed link 1146
- removed link 1147
- removed link 22
- removed link 224
- removed link 348
- removed link 352
- removed link 410
- removed link 417
- removed link 425
- removed link 43
- removed link 432
- removed link 439
- removed link 556
- removed link 560
- removed link 611
- removed link 613
- removed link 615
- removed link 618
- removed link 620
- removed link 622
- removed link 626
- removed link 628
- removed link 630
- removed link 633
- removed link 635
- removed link 637
- removed link 64
- removed link 640
- removed link 642
- removed link 644
- removed link 66
- removed link 68
- removed link 764
- removed link 812
- removed link 814
- removed link 816
- removed link 819
- removed link 821
- removed link 823
- removed link 827
- removed link 829
- removed link 831
- removed link 834
- removed link 836
- removed link 838
- removed link 841
- removed link 843
- removed link 845
- removed link 85
- removed link 87
- removed link 89
- removed link 957
- removed link 958
- removed link 959
- removed link 961
- removed link 962
- removed link 963
- link 0: mass 0.8139458541752262 -> 0.1266493789566258; geometry collision cylinder length=1.2050055825401313 radius=0.18290773275572914; visual cylinder length=1.2050055825401313 radius=0.18290773275572914
Joints:
- removed joint 1049_to_348
- removed joint 1050_to_348
- removed joint 1051_to_348
- removed joint 1053_to_352
- removed joint 1054_to_352
- removed joint 1055_to_352
- removed joint 1146_to_11
- removed joint 1147_to_11
- removed joint 11_to_0
- removed joint 224_to_11
- removed joint 22_to_11
- removed joint 348_to_0
- removed joint 352_to_0
- removed joint 410_to_22
- removed joint 417_to_22
- removed joint 425_to_224
- removed joint 432_to_224
- removed joint 439_to_224
- removed joint 43_to_22
- removed joint 556_to_0
- removed joint 560_to_0
- removed joint 611_to_410
- removed joint 613_to_410
- removed joint 615_to_410
- removed joint 618_to_417
- removed joint 620_to_417
- removed joint 622_to_417
- removed joint 626_to_425
- removed joint 628_to_425
- removed joint 630_to_425
- removed joint 633_to_432
- removed joint 635_to_432
- removed joint 637_to_432
- removed joint 640_to_439
- removed joint 642_to_439
- removed joint 644_to_439
- removed joint 64_to_43
- removed joint 66_to_43
- removed joint 68_to_43
- removed joint 764_to_0
- removed joint 812_to_611
- removed joint 814_to_613
- removed joint 816_to_615
- removed joint 819_to_618
- removed joint 821_to_620
- removed joint 823_to_622
- removed joint 827_to_626
- removed joint 829_to_628
- removed joint 831_to_630
- removed joint 834_to_633
- removed joint 836_to_635
- removed joint 838_to_637
- removed joint 841_to_640
- removed joint 843_to_642
- removed joint 845_to_644
- removed joint 85_to_64
- removed joint 87_to_66
- removed joint 89_to_68
- removed joint 957_to_556
- removed joint 958_to_556
- removed joint 959_to_556
- removed joint 961_to_560
- removed joint 962_to_560
- removed joint 963_to_560

File: temp7.urdf (robot description, URDF)
Before this commit: robot pepe, 85 links, 84 joints
Links:
- removed link 1027
- removed link 1028
- removed link 1032
- removed link 1033
- removed link 1037
- removed link 1038
- removed link 1067
- removed link 1068
- removed link 1072
- removed link 1073
- removed link 1077
- removed link 1078
- removed link 1182
- removed link 1183
- removed link 1184
- removed link 22
- removed link 242
- removed link 310
- removed link 317
- removed link 33
- removed link 343
- removed link 350
- removed link 357
- removed link 424
- removed link 429
- removed link 434
- removed link 464
- removed link 469
- removed link 474
- removed link 511
- removed link 512
- removed link 513
- removed link 518
- removed link 519
- removed link 520
- removed link 54
- removed link 544
- removed link 545
- removed link 546
- removed link 55
- removed link 551
- removed link 552
- removed link 553
- removed link 558
- removed link 559
- removed link 56
- removed link 560
- removed link 625
- removed link 630
- removed link 635
- removed link 665
- removed link 670
- removed link 675
- removed link 739
- removed link 740
- removed link 741
- removed link 779
- removed link 780
- removed link 781
- removed link 826
- removed link 831
- removed link 836
- removed link 866
- removed link 871
- removed link 876
- removed link 914
- removed link 915
- removed link 916
- removed link 921
- removed link 922
- removed link 923
- removed link 947
- removed link 948
- removed link 949
- removed link 954
- removed link 955
- removed link 956
- removed link 961
- removed link 962
- removed link 963
- removed link 97
- removed link 98
- removed link 99
- link 0: mass 0.0002810120252331259 -> 0.1266493789566258; geometry collision cylinder length=1.2050055825401313 radius=0.18290773275572914; visual cylinder length=1.2050055825401313 radius=0.18290773275572914
- link 11: mass 0.9729272846353406 -> 2.561384175740279; geometry collision cylinder length=0.8154769926966201 radius=0.9999; visual cylinder length=0.8154769926966201 radius=0.9999
Joints:
- removed joint 1027_to_424
- removed joint 1028_to_424
- removed joint 1032_to_429
- removed joint 1033_to_429
- removed joint 1037_to_434
- removed joint 1038_to_434
- removed joint 1067_to_464
- removed joint 1068_to_464
- removed joint 1072_to_469
- removed joint 1073_to_469
- removed joint 1077_to_474
- removed joint 1078_to_474
- removed joint 1182_to_0
- removed joint 1183_to_0
- removed joint 1184_to_0
- removed joint 22_to_11
- removed joint 242_to_11
- removed joint 310_to_22
- removed joint 317_to_22
- removed joint 33_to_22
- removed joint 343_to_242
- removed joint 350_to_242
- removed joint 357_to_242
- removed joint 424_to_22
- removed joint 429_to_22
- removed joint 434_to_22
- removed joint 464_to_242
- removed joint 469_to_242
- removed joint 474_to_242
- removed joint 511_to_310
- removed joint 512_to_310
- removed joint 513_to_310
- removed joint 518_to_317
- removed joint 519_to_317
- removed joint 520_to_317
- removed joint 544_to_343
- removed joint 545_to_343
- removed joint 546_to_343
- removed joint 54_to_33
- removed joint 551_to_350
- removed joint 552_to_350
- removed joint 553_to_350
- removed joint 558_to_357
- removed joint 559_to_357
- removed joint 55_to_33
- removed joint 560_to_357
- removed joint 56_to_33
- removed joint 625_to_424
- removed joint 630_to_429
- removed joint 635_to_434
- removed joint 665_to_464
- removed joint 670_to_469
- removed joint 675_to_474
- removed joint 739_to_22
- removed joint 740_to_22
- removed joint 741_to_22
- removed joint 779_to_242
- removed joint 780_to_242
- removed joint 781_to_242
- removed joint 826_to_424
- removed joint 831_to_429
- removed joint 836_to_434
- removed joint 866_to_464
- removed joint 871_to_469
- removed joint 876_to_474
- removed joint 914_to_310
- removed joint 915_to_310
- removed joint 916_to_310
- removed joint 921_to_317
- removed joint 922_to_317
- removed joint 923_to_317
- removed joint 947_to_343
- removed joint 948_to_343
- removed joint 949_to_343
- removed joint 954_to_350
- removed joint 955_to_350
- removed joint 956_to_350
- removed joint 961_to_357
- removed joint 962_to_357
- removed joint 963_to_357
- removed joint 97_to_33
- removed joint 98_to_33
- removed joint 99_to_33
- joint 11_to_0: origin xyz=0.7552850851251348 0.5012198787045238 0.928150598676136 rpy=8.547940858668197 1.0149326589339163 2.9253246612287014 -> xyz=0.5488228574833086 0.6727352694338915 0.9999 rpy=9.187154749586885 4.526911794548183 5.196853465412705

Commit message: rollback wrong params in exp pop_size

File: temp0.urdf (robot description, URDF)
Before this commit: robot pepe, 2 links, 1 joints
Links:
- added link 12, mass 5.831947733639437; collision cylinder length=1.856737948346875 radius=0.9999; visual cylinder length=1.856737948346875 radius=0.9999
- link 0: mass 0.1266493789566258 -> 0.4629260655908738; geometry collision cylinder length=0.7967607353490778 radius=0.43004798710737613; visual cylinder length=0.7967607353490778 radius=0.43004798710737613
- link 11: mass 2.561384175740279 -> 5.831947733639437; geometry collision cylinder length=1.856737948346875 radius=0.9999; visual cylinder length=1.856737948346875 radius=0.9999
Joints:
- added joint 12_to_0: type revolute, parent 0, child 12, origin xyz=0.9921446809327699 0.9999 0.7039010056764574 rpy=18.847670965946605 5.358322996685524 1.1143862440410601, axis 1 0 0, limit lower=3.1415 upper=-3.1415 effort=1 velocity=1
- joint 11_to_0: axis 0 1 0 -> 1 0 0; origin xyz=0.5488228574833086 0.7727352694338915 0.9999 rpy=9.187154749586885 4.526911794548183 5.196853465412705 -> xyz=0.9921446809327699 0.9999 0.7039010056764574 rpy=12.565113977297736 5.358322996685524 1.1143862440410601

File: temp1.urdf (robot description, URDF)
Before this commit: robot pepe, 4 links, 3 joints
Links:
- removed link 13
- link 0: mass 2.561384175740279 -> 5.831947733639437; geometry collision cylinder length=1.856737948346875 radius=0.9999; visual cylinder length=1.856737948346875 radius=0.9999
- link 11: mass 0.1266493789566258 -> 5.831947733639437; geometry collision cylinder length=1.856737948346875 radius=0.9999; visual cylinder length=1.856737948346875 radius=0.9999
- link 12: mass 0.1266493789566258 -> 5.831947733639437; geometry collision cylinder length=1.856737948346875 radius=0.9999; visual cylinder length=1.856737948346875 radius=0.9999
Joints:
- removed joint 13_to_0
- joint 11_to_0: axis 0 1 0 -> 1 0 0; origin xyz=0.29548778666124453 0.12065575549339036 0.5154713031273903 rpy=4.9167587414661424 4.924491704359826 3.0762963088839346 -> xyz=0.9921446809327699 0.9999 0.8039010056764574 rpy=12.565113977297736 5.358322996685524 1.1143862440410601
- joint 12_to_0: axis 0 1 0 -> 1 0 0; origin xyz=0.29548778666124453 0.12065575549339036 0.5154713031273903 rpy=7.375138112199213 4.924491704359826 3.0762963088839346 -> xyz=0.9921446809327699 0.9999 0.8039010056764574 rpy=18.847670965946605 5.358322996685524 1.1143862440410601

File: temp2.urdf (robot description, URDF)
Before this commit: robot pepe, 1 links, 0 joints
Links:
- added link 11, mass 0.879774102452685; collision cylinder length=0.9967607353490777 radius=0.5300479871073761; visual cylinder length=0.9967607353490777 radius=0.5300479871073761
- link 0: mass 2.6568424106949546 -> 2.3124693735144346; geometry collision cylinder length=1.149073549002775 radius=0.8003669461604143; visual cylinder length=1.149073549002775 radius=0.8003669461604143
Joints:
- added joint 11_to_0: type revolute, parent 0, child 11, origin xyz=0.9999 0.6524380266579504 0.6067726166371412 rpy=8.254602059531974 4.674758863147256 1.4498086777749795, axis 0 0 1, limit lower=3.1415 upper=-3.1415 effort=1 velocity=1

File: temp3.urdf (robot description, URDF)
Before this commit: robot pepe, 1 links, 0 joints
Links:
- added link 11, mass 2.3124693735144346; collision cylinder length=1.149073549002775 radius=0.8003669461604143; visual cylinder length=1.149073549002775 radius=0.8003669461604143
- added link 12, mass 2.3124693735144346; collision cylinder length=1.149073549002775 radius=0.8003669461604143; visual cylinder length=1.149073549002775 radius=0.8003669461604143
- added link 13, mass 2.3124693735144346; collision cylinder length=1.149073549002775 radius=0.8003669461604143; visual cylinder length=1.149073549002775 radius=0.8003669461604143
- link 0: mass 2.561384175740279 -> 6.281300540076709; geometry collision cylinder length=1.9998 radius=0.9999; visual cylinder length=1.9998 radius=0.9999
Joints:
- added joint 11_to_0: type revolute, parent 0, child 11, origin xyz=0.7366060435001854 0.2904574810689805 0.7492643203752772 rpy=6.988460235719735 2.860661912110513 1.3541356266205908, axis 1 0 0, limit lower=3.1415 upper=-3.1415 effort=1 velocity=1
- added joint 12_to_0: type revolute, parent 0, child 12, origin xyz=0.7366060435001854 0.2904574810689805 0.7492643203752772 rpy=10.482690353579603 2.860661912110513 1.3541356266205908, axis 1 0 0, limit lower=3.1415 upper=-3.1415 effort=1 velocity=1
- added joint 13_to_0: type revolute, parent 0, child 13, origin xyz=0.7366060435001854 0.2904574810689805 0.7492643203752772 rpy=13.97692047143947 2.860661912110513 1.3541356266205908, axis 1 0 0, limit lower=3.1415 upper=-3.1415 effort=1 velocity=1

File: temp4.urdf (robot description, URDF)
Before this commit: robot pepe, 2 links, 1 joints
Links:
- link 0: mass 0.1266493789566258 -> 0.4629260655908738; geometry collision cylinder length=0.7967607353490778 radius=0.43004798710737613; visual cylinder length=0.7967607353490778 radius=0.43004798710737613
- link 11: mass 2.561384175740279 -> 1.492466052373412; geometry collision cylinder length=1.1967607353490777 radius=0.6300479871073761; visual cylinder length=1.1967607353490777 radius=0.6300479871073761
Joints:
- joint 11_to_0: axis 0 1 0 -> 0 0 1; origin xyz=0.5488228574833086 0.6727352694338915 0.9037495979989713 rpy=9.187154749586885 4.526911794548183 5.196853465412705 -> xyz=0.9999 0.7524380266579503 0.9067726166371411 rpy=6.997964998096057 5.931395924583172 3.3347642699288556

File: temp5.urdf (robot description, URDF)
Before this commit: robot pepe, 1 links, 0 joints
Links:
- added link 11, mass 0.4629260655908738; collision cylinder length=0.7967607353490778 radius=0.43004798710737613; visual cylinder length=0.7967607353490778 radius=0.43004798710737613
- added link 22, mass 5.831947733639437; collision cylinder length=1.856737948346875 radius=0.9999; visual cylinder length=1.856737948346875 radius=0.9999
- added link 25, mass 5.831947733639437; collision cylinder length=1.856737948346875 radius=0.9999; visual cylinder length=1.856737948346875 radius=0.9999
- added link 33, mass 0.12781138190273833; collision cylinder length=1.2924712818558965 radius=0.17741869393731358; visual cylinder length=1.2924712818558965 radius=0.17741869393731358
- added link 34, mass 0.12781138190273833; collision cylinder length=1.2924712818558965 radius=0.17741869393731358; visual cylinder length=1.2924712818558965 radius=0.17741869393731358
- added link 36, mass 0.12781138190273833; collision cylinder length=1.2924712818558965 radius=0.17741869393731358; visual cylinder length=1.2924712818558965 radius=0.17741869393731358
- added link 37, mass 0.12781138190273833; collision cylinder length=1.2924712818558965 radius=0.17741869393731358; visual cylinder length=1.2924712818558965 radius=0.17741869393731358
- link 0: mass 2.1335725720273833 -> 2.714962212292477; geometry collision cylinder length=1.349073549002775 radius=0.8003669461604143; visual cylinder length=1.349073549002775 radius=0.8003669461604143
Joints:
- added joint 11_to_0: type revolute, parent 0, child 11, origin xyz=0.9563592729508589 0.6524380266579504 0.6067726166371412 rpy=6.997964998096057 4.674758863147256 1.4498086777749795, axis 0 0 1, limit lower=3.1415 upper=-3.1415 effort=1 velocity=1
- added joint 22_to_11: type revolute, parent 11, child 22, origin xyz=0.9921446809327699 0.9999 0.7039010056764574 rpy=12.565113977297736 5.358322996685524 1.1143862440410601, axis 1 0 0, limit lower=3.1415 upper=-3.1415 effort=1 velocity=1
- added joint 25_to_11: type revolute, parent 11, child 25, origin xyz=0.9921446809327699 0.9999 0.7039010056764574 rpy=18.847670965946605 5.358322996685524 1.1143862440410601, axis 1 0 0, limit lower=3.1415 upper=-3.1415 effort=1 velocity=1
- added joint 33_to_22: type revolute, parent 22, child 33, origin xyz=0.7677225202684853 0.7526722238192851 0.8568453700284847 rpy=2.0556543177386426 4.786743107309758 1.4581030541810585, axis 0 0 1, limit lower=3.1415 upper=-3.1415 effort=1 velocity=1
- added joint 34_to_22: type revolute, parent 22, child 34, origin xyz=0.7677225202684853 0.7526722238192851 0.8568453700284847 rpy=3.0834814766079637 4.786743107309758 1.4581030541810585, axis 0 0 1, limit lower=3.1415 upper=-3.1415 effort=1 velocity=1
- added joint 36_to_25: type revolute, parent 25, child 36, origin xyz=0.7677225202684853 0.7526722238192851 0.8568453700284847 rpy=2.0556543177386426 4.786743107309758 1.4581030541810585, axis 0 0 1, limit lower=3.1415 upper=-3.1415 effort=1 velocity=1
- added joint 37_to_25: type revolute, parent 25, child 37, origin xyz=0.7677225202684853 0.7526722238192851 0.8568453700284847 rpy=3.0834814766079637 4.786743107309758 1.4581030541810585, axis 0 0 1, limit lower=3.1415 upper=-3.1415 effort=1 velocity=1

File: temp6.urdf (robot description, URDF)
Before this commit: robot pepe, 1 links, 0 joints
Links:
- added link 11, mass 1.492466052373412; collision cylinder length=1.1967607353490777 radius=0.6300479871073761; visual cylinder length=1.1967607353490777 radius=0.6300479871073761
- link 0: mass 0.1266493789566258 -> 0.6953301211888475; geometry collision cylinder length=1.1967607353490777 radius=0.43004798710737613; visual cylinder length=1.1967607353490777 radius=0.43004798710737613
Joints:
- added joint 11_to_0: type revolute, parent 0, child 11, origin xyz=0.9999 0.8524380266579503 0.9067726166371411 rpy=6.997964998096057 5.931395924583172 3.3347642699288556, axis 0 0 1, limit lower=3.1415 upper=-3.1415 effort=1 velocity=1

File: temp7.urdf (robot description, URDF)
Before this commit: robot pepe, 2 links, 1 joints
Links:
- removed link 11
- link 0: mass 0.1266493789566258 -> 0.4629260655908738; geometry collision cylinder length=0.7967607353490778 radius=0.43004798710737613; visual cylinder length=0.7967607353490778 radius=0.43004798710737613
Joints:
- removed joint 11_to_0
