Commit message: fix typo in csv

File: temp0.urdf (robot description, URDF)
Before this commit: robot pepe, 3 links, 2 joints
Links:
- added link 13, mass 0.1741890424965086; collision cylinder length=0.9274469940070369 radius=0.24450679369046097; visual cylinder length=0.9274469940070369 radius=0.24450679369046097
- link 0: mass 0.4629260655908738 -> 6.281300540076709; geometry collision cylinder length=1.9998 radius=0.9999; visual cylinder length=1.9998 radius=0.9999
- link 11: mass 5.831947733639437 -> 0.1741890424965086; geometry collision cylinder length=0.9274469940070369 radius=0.24450679369046097; visual cylinder length=0.9274469940070369 radius=0.24450679369046097
- link 12: mass 5.831947733639437 -> 0.1741890424965086; geometry collision cylinder length=0.9274469940070369 radius=0.24450679369046097; visual cylinder length=0.9274469940070369 radius=0.24450679369046097
Joints:
- added joint 13_to_0: type revolute, parent 0, child 13, origin xyz=0.5507040907358064 0.3018865040146698 0.2808948815863546 rpy=25.00280673805323 6.282556988648868 4.095839754883953, axis 0 0 1, limit lower=3.1415 upper=-3.1415 effort=1 velocity=1
- joint 11_to_0: axis 1 0 0 -> 0 0 1; origin xyz=0.9921446809327699 0.9999 0.7039010056764574 rpy=12.565113977297736 5.358322996685524 1.1143862440410601 -> xyz=0.5507040907358064 0.3018865040146698 0.2808948815863546 rpy=12.501403369026615 6.282556988648868 4.095839754883953
- joint 12_to_0: axis 1 0 0 -> 0 0 1; origin xyz=0.9921446809327699 0.9999 0.7039010056764574 rpy=18.847670965946605 5.358322996685524 1.1143862440410601 -> xyz=0.5507040907358064 0.3018865040146698 0.2808948815863546 rpy=18.75210505353992 6.282556988648868 4.095839754883953

File: temp1.urdf (robot description, URDF)
Before this commit: robot pepe, 3 links, 2 joints
Links:
- removed link 11
- removed link 12
- link 0: mass 5.831947733639437 -> 4.666439726850212; geometry collision cylinder length=1.4856710176840369 radius=0.9999; visual cylinder length=1.4856710176840369 radius=0.9999
Joints:
- removed joint 11_to_0
- removed joint 12_to_0

File: temp2.urdf (robot description, URDF)
Before this commit: robot pepe, 2 links, 1 joints
Links:
- added link 12, mass 5.922825473440213; collision cylinder length=1.8856710176840368 radius=0.9999; visual cylinder length=1.8856710176840368 radius=0.9999
- added link 13, mass 5.922825473440213; collision cylinder length=1.8856710176840368 radius=0.9999; visual cylinder length=1.8856710176840368 radius=0.9999
- link 0: mass 2.3124693735144346 -> 6.281300540076709; geometry collision cylinder length=1.9998 radius=0.9999; visual cylinder length=1.9998 radius=0.9999
- link 11: mass 0.879774102452685 -> 5.922825473440213; geometry collision cylinder length=1.8856710176840368 radius=0.9999; visual cylinder length=1.8856710176840368 radius=0.9999
Joints:
- added joint 12_to_0: type revolute, parent 0, child 12, origin xyz=0.9999 0.9999 0.9999 rpy=17.18453429315246 6.282556988648868 6.282556988648868, axis 0 0 1, limit lower=3.1415 upper=-3.1415 effort=1 velocity=1
- added joint 13_to_0: type revolute, parent 0, child 13, origin xyz=0.9999 0.9999 0.9999 rpy=22.912712390869945 6.282556988648868 6.282556988648868, axis 0 0 1, limit lower=3.1415 upper=-3.1415 effort=1 velocity=1
- joint 11_to_0: origin xyz=0.9999 0.6524380266579504 0.6067726166371412 rpy=8.254602059531974 4.674758863147256 1.4498086777749795 -> xyz=0.9999 0.9999 0.9999 rpy=11.456356195434973 6.282556988648868 6.282556988648868

File: temp3.urdf (robot description, URDF)
Before this commit: robot pepe, 4 links, 3 joints
Links:
- removed link 11
- removed link 12
- removed link 13
- link 0: mass 6.281300540076709 -> 4.666439726850212; geometry collision cylinder length=1.4856710176840369 radius=0.9999; visual cylinder length=1.4856710176840369 radius=0.9999
Joints:
- removed joint 11_to_0
- removed joint 12_to_0
- removed joint 13_to_0

File: temp4.urdf (robot description, URDF)
Before this commit: robot pepe, 2 links, 1 joints
Links:
- added link 12, mass 5.922825473440213; collision cylinder length=1.8856710176840368 radius=0.9999; visual cylinder length=1.8856710176840368 radius=0.9999
- added link 13, mass 5.922825473440213; collision cylinder length=1.8856710176840368 radius=0.9999; visual cylinder length=1.8856710176840368 radius=0.9999
- link 0: mass 0.4629260655908738 -> 3.4100539802602117; geometry collision cylinder length=1.085671017684037 radius=0.9999; visual cylinder length=1.085671017684037 radius=0.9999
- link 11: mass 1.492466052373412 -> 5.922825473440213; geometry collision cylinder length=1.8856710176840368 radius=0.9999; visual cylinder length=1.8856710176840368 radius=0.9999
Joints:
- added joint 12_to_0: type revolute, parent 0, child 12, origin xyz=0.9999 0.9999 0.9999 rpy=13.414623108844708 6.282556988648868 6.282556988648868, axis 0 0 1, limit lower=3.1415 upper=-3.1415 effort=1 velocity=1
- added joint 13_to_0: type revolute, parent 0, child 13, origin xyz=0.9999 0.9999 0.9999 rpy=17.886164145126276 6.282556988648868 6.282556988648868, axis 0 0 1, limit lower=3.1415 upper=-3.1415 effort=1 velocity=1
- joint 11_to_0: origin xyz=0.9999 0.7524380266579503 0.9067726166371411 rpy=6.997964998096057 5.931395924583172 3.3347642699288556 -> xyz=0.9999 0.9999 0.9999 rpy=8.943082072563138 6.282556988648868 6.282556988648868

File: temp5.urdf (robot description, URDF)
Before this commit: robot pepe, 8 links, 7 joints
Links:
- removed link 22
- removed link 25
- removed link 33
- removed link 34
- removed link 36
- removed link 37
- added link 12, mass 5.922825473440213; collision cylinder length=1.8856710176840368 radius=0.9999; visual cylinder length=1.8856710176840368 radius=0.9999
- added link 13, mass 5.922825473440213; collision cylinder length=1.8856710176840368 radius=0.9999; visual cylinder length=1.8856710176840368 radius=0.9999
- link 0: mass 2.714962212292477 -> 3.4100539802602117; geometry collision cylinder length=1.085671017684037 radius=0.9999; visual cylinder length=1.085671017684037 radius=0.9999
- link 11: mass 0.4629260655908738 -> 5.922825473440213; geometry collision cylinder length=1.8856710176840368 radius=0.9999; visual cylinder length=1.8856710176840368 radius=0.9999
Joints:
- removed joint 22_to_11
- removed joint 25_to_11
- removed joint 33_to_22
- removed joint 34_to_22
- removed joint 36_to_25
- removed joint 37_to_25
- added joint 12_to_0: type revolute, parent 0, child 12, origin xyz=0.9999 0.9999 0.9999 rpy=13.414623108844708 6.282556988648868 6.282556988648868, axis 0 0 1, limit lower=3.1415 upper=-3.1415 effort=1 velocity=1
- added joint 13_to_0: type revolute, parent 0, child 13, origin xyz=0.9999 0.9999 0.9999 rpy=17.886164145126276 6.282556988648868 6.282556988648868, axis 0 0 1, limit lower=3.1415 upper=-3.1415 effort=1 velocity=1
- joint 11_to_0: origin xyz=0.9563592729508589 0.6524380266579504 0.6067726166371412 rpy=6.997964998096057 4.674758863147256 1.4498086777749795 -> xyz=0.9999 0.9999 0.9999 rpy=8.943082072563138 6.282556988648868 6.282556988648868

File: temp6.urdf (robot description, URDF)
Before this commit: robot pepe, 2 links, 1 joints
Links:
- added link 12, mass 4.038246853555211; collision cylinder length=1.285671017684037 radius=0.9999; visual cylinder length=1.285671017684037 radius=0.9999
- added link 13, mass 4.038246853555211; collision cylinder length=1.285671017684037 radius=0.9999; visual cylinder length=1.285671017684037 radius=0.9999
- link 0: mass 0.6953301211888475 -> 3.4100539802602117; geometry collision cylinder length=1.085671017684037 radius=0.9999; visual cylinder length=1.085671017684037 radius=0.9999
- link 11: mass 1.492466052373412 -> 4.038246853555211; geometry collision cylinder length=1.285671017684037 radius=0.9999; visual cylinder length=1.285671017684037 radius=0.9999
Joints:
- added joint 12_to_0: type revolute, parent 0, child 12, origin xyz=0.9999 0.9500845945394578 0.9999 rpy=9.644711924536956 3.8001087162635065 5.976593086836112, axis 0 0 1, limit lower=3.1415 upper=-3.1415 effort=1 velocity=1
- added joint 13_to_0: type revolute, parent 0, child 13, origin xyz=0.9999 0.9500845945394578 0.9999 rpy=12.859615899382609 3.8001087162635065 5.976593086836112, axis 0 0 1, limit lower=3.1415 upper=-3.1415 effort=1 velocity=1
- joint 11_to_0: origin xyz=0.9999 0.8524380266579503 0.9067726166371411 rpy=6.997964998096057 5.931395924583172 3.3347642699288556 -> xyz=0.9999 0.9500845945394578 0.9999 rpy=6.4298079496913045 3.8001087162635065 5.976593086836112

File: temp7.urdf (robot description, URDF)
Before this commit: robot pepe, 1 links, 0 joints
Links:
- added link 11, mass 0.4203795558477106; collision cylinder length=1.1274469940070369 radius=0.344506793690461; visual cylinder length=1.1274469940070369 radius=0.344506793690461
- added link 12, mass 0.4203795558477106; collision cylinder length=1.1274469940070369 radius=0.344506793690461; visual cylinder length=1.1274469940070369 radius=0.344506793690461
- added link 13, mass 0.4203795558477106; collision cylinder length=1.1274469940070369 radius=0.344506793690461; visual cylinder length=1.1274469940070369 radius=0.344506793690461
- link 0: mass 0.4629260655908738 -> 5.922825473440213; geometry collision cylinder length=1.8856710176840368 radius=0.9999; visual cylinder length=1.8856710176840368 radius=0.9999
Joints:
- added joint 11_to_0: type revolute, parent 0, child 11, origin xyz=0.5507040907358064 0.5018865040146698 0.48089488158635463 rpy=12.565113977297736 6.282556988648868 5.352476816319871, axis 0 0 1, limit lower=3.1415 upper=-3.1415 effort=1 velocity=1
- added joint 12_to_0: type revolute, parent 0, child 12, origin xyz=0.5507040907358064 0.5018865040146698 0.48089488158635463 rpy=18.847670965946605 6.282556988648868 5.352476816319871, axis 0 0 1, limit lower=3.1415 upper=-3.1415 effort=1 velocity=1
- added joint 13_to_0: type revolute, parent 0, child 13, origin xyz=0.5507040907358064 0.5018865040146698 0.48089488158635463 rpy=25.130227954595473 6.282556988648868 5.352476816319871, axis 0 0 1, limit lower=3.1415 upper=-3.1415 effort=1 velocity=1
