Commit message: genome spec experiments

File: temp0.urdf (robot description, URDF)
Before this commit: robot pepe, 4 links, 3 joints
Links:
- added link 14, mass 0.06629730966755146; collision cylinder length=0.8600601898436186 radius=0.15664213484259137; visual cylinder length=0.8600601898436186 radius=0.15664213484259137
- added link 15, mass 0.06629730966755146; collision cylinder length=0.8600601898436186 radius=0.15664213484259137; visual cylinder length=0.8600601898436186 radius=0.15664213484259137
- link 0: mass 6.281300540076709 -> 4.858362961097827; geometry collision cylinder length=1.5467743005789663 radius=0.9999; visual cylinder length=1.5467743005789663 radius=0.9999
- link 11: mass 0.1741890424965086 -> 0.06629730966755146; geometry collision cylinder length=0.8600601898436186 radius=0.15664213484259137; visual cylinder length=0.8600601898436186 radius=0.15664213484259137
- link 12: mass 0.1741890424965086 -> 0.06629730966755146; geometry collision cylinder length=0.8600601898436186 radius=0.15664213484259137; visual cylinder length=0.8600601898436186 radius=0.15664213484259137
- link 13: mass 0.1741890424965086 -> 0.06629730966755146; geometry collision cylinder length=0.8600601898436186 radius=0.15664213484259137; visual cylinder length=0.8600601898436186 radius=0.15664213484259137
Joints:
- added joint 14_to_0: type revolute, parent 0, child 14, origin xyz=0.8917763905858218 0.986858241253344 0.6929518411048576 rpy=26.744218351542326 4.953343961282325 5.190068367303865, axis 1 0 0, limit lower=3.1415 upper=-3.1415 effort=1 velocity=1
- added joint 15_to_0: type revolute, parent 0, child 15, origin xyz=0.8917763905858218 0.986858241253344 0.6929518411048576 rpy=32.09306202185079 4.953343961282325 5.190068367303865, axis 1 0 0, limit lower=3.1415 upper=-3.1415 effort=1 velocity=1
- joint 11_to_0: axis 0 0 1 -> 1 0 0; origin xyz=0.5507040907358064 0.3018865040146698 0.2808948815863546 rpy=12.501403369026615 6.282556988648868 4.095839754883953 -> xyz=0.8917763905858218 0.986858241253344 0.6929518411048576 rpy=10.69768734061693 4.953343961282325 5.190068367303865
- joint 12_to_0: axis 0 0 1 -> 1 0 0; origin xyz=0.5507040907358064 0.3018865040146698 0.2808948815863546 rpy=18.75210505353992 6.282556988648868 4.095839754883953 -> xyz=0.8917763905858218 0.986858241253344 0.6929518411048576 rpy=16.046531010925396 4.953343961282325 5.190068367303865
- joint 13_to_0: axis 0 0 1 -> 1 0 0; origin xyz=0.5507040907358064 0.3018865040146698 0.2808948815863546 rpy=25.00280673805323 6.282556988648868 4.095839754883953 -> xyz=0.8917763905858218 0.986858241253344 0.6929518411048576 rpy=21.39537468123386 4.953343961282325 5.190068367303865

File: temp1.urdf (robot description, URDF)
Before this commit: robot pepe, 1 links, 0 joints
Links:
- added link 11, mass 0.23124444030073726; collision cylinder length=1.2375544128684464 radius=0.24388133411571777; visual cylinder length=1.2375544128684464 radius=0.24388133411571777
- added link 110, mass 0.23124444030073726; collision cylinder length=1.2375544128684464 radius=0.24388133411571777; visual cylinder length=1.2375544128684464 radius=0.24388133411571777
- added link 119, mass 0.23124444030073726; collision cylinder length=1.2375544128684464 radius=0.24388133411571777; visual cylinder length=1.2375544128684464 radius=0.24388133411571777
- added link 211, mass 0.10350372323662803; collision cylinder length=1.2116260460477128 radius=0.16489927627096637; visual cylinder length=1.2116260460477128 radius=0.16489927627096637
- added link 212, mass 0.10350372323662803; collision cylinder length=1.2116260460477128 radius=0.16489927627096637; visual cylinder length=1.2116260460477128 radius=0.16489927627096637
- added link 213, mass 0.10350372323662803; collision cylinder length=1.2116260460477128 radius=0.16489927627096637; visual cylinder length=1.2116260460477128 radius=0.16489927627096637
- added link 22, mass 0.10350372323662803; collision cylinder length=1.2116260460477128 radius=0.16489927627096637; visual cylinder length=1.2116260460477128 radius=0.16489927627096637
- added link 220, mass 0.10350372323662803; collision cylinder length=1.2116260460477128 radius=0.16489927627096637; visual cylinder length=1.2116260460477128 radius=0.16489927627096637
- added link 221, mass 0.10350372323662803; collision cylinder length=1.2116260460477128 radius=0.16489927627096637; visual cylinder length=1.2116260460477128 radius=0.16489927627096637
- added link 222, mass 0.10350372323662803; collision cylinder length=1.2116260460477128 radius=0.16489927627096637; visual cylinder length=1.2116260460477128 radius=0.16489927627096637
- added link 23, mass 0.10350372323662803; collision cylinder length=1.2116260460477128 radius=0.16489927627096637; visual cylinder length=1.2116260460477128 radius=0.16489927627096637
- added link 24, mass 0.10350372323662803; collision cylinder length=1.2116260460477128 radius=0.16489927627096637; visual cylinder length=1.2116260460477128 radius=0.16489927627096637
- added link 314, mass 2.313001156161996; collision cylinder length=1.5219057551912725 radius=0.6955351920275803; visual cylinder length=1.5219057551912725 radius=0.6955351920275803
- added link 315, mass 2.313001156161996; collision cylinder length=1.5219057551912725 radius=0.6955351920275803; visual cylinder length=1.5219057551912725 radius=0.6955351920275803
- added link 316, mass 2.313001156161996; collision cylinder length=1.5219057551912725 radius=0.6955351920275803; visual cylinder length=1.5219057551912725 radius=0.6955351920275803
- added link 317, mass 2.313001156161996; collision cylinder length=1.5219057551912725 radius=0.6955351920275803; visual cylinder length=1.5219057551912725 radius=0.6955351920275803
- added link 318, mass 2.313001156161996; collision cylinder length=1.5219057551912725 radius=0.6955351920275803; visual cylinder length=1.5219057551912725 radius=0.6955351920275803
- added link 323, mass 2.313001156161996; collision cylinder length=1.5219057551912725 radius=0.6955351920275803; visual cylinder length=1.5219057551912725 radius=0.6955351920275803
- added link 324, mass 2.313001156161996; collision cylinder length=1.5219057551912725 radius=0.6955351920275803; visual cylinder length=1.5219057551912725 radius=0.6955351920275803
- added link 325, mass 2.313001156161996; collision cylinder length=1.5219057551912725 radius=0.6955351920275803; visual cylinder length=1.5219057551912725 radius=0.6955351920275803
- added link 326, mass 2.313001156161996; collision cylinder length=1.5219057551912725 radius=0.6955351920275803; visual cylinder length=1.5219057551912725 radius=0.6955351920275803
- added link 327, mass 2.313001156161996; collision cylinder length=1.5219057551912725 radius=0.6955351920275803; visual cylinder length=1.5219057551912725 radius=0.6955351920275803
- added link 35, mass 2.313001156161996; collision cylinder length=1.5219057551912725 radius=0.6955351920275803; visual cylinder length=1.5219057551912725 radius=0.6955351920275803
- added link 36, mass 2.313001156161996; collision cylinder length=1.5219057551912725 radius=0.6955351920275803; visual cylinder length=1.5219057551912725 radius=0.6955351920275803
- added link 37, mass 2.313001156161996; collision cylinder length=1.5219057551912725 radius=0.6955351920275803; visual cylinder length=1.5219057551912725 radius=0.6955351920275803
- added link 38, mass 2.313001156161996; collision cylinder length=1.5219057551912725 radius=0.6955351920275803; visual cylinder length=1.5219057551912725 radius=0.6955351920275803
- added link 39, mass 2.313001156161996; collision cylinder length=1.5219057551912725 radius=0.6955351920275803; visual cylinder length=1.5219057551912725 radius=0.6955351920275803
- link 0: mass 4.666439726850212 -> 4.858362961097827; geometry collision cylinder length=1.5467743005789663 radius=0.9999; visual cylinder length=1.5467743005789663 radius=0.9999
Joints:
- added joint 110_to_0: type revolute, parent 0, child 110, origin xyz=0.14202291316859839 0.4886344072576644 0.8976997633809118 rpy=16.435411072782838 0.7190774033016101 0.2733466792329027, axis 0 0 1, limit lower=3.1415 upper=-3.1415 effort=1 velocity=1
- added joint 119_to_0: type revolute, parent 0, child 119, origin xyz=0.14202291316859839 0.4886344072576644 0.8976997633809118 rpy=21.913881430377117 0.7190774033016101 0.2733466792329027, axis 0 0 1, limit lower=3.1415 upper=-3.1415 effort=1 velocity=1
- added joint 11_to_0: type revolute, parent 0, child 11, origin xyz=0.14202291316859839 0.4886344072576644 0.8976997633809118 rpy=10.956940715188558 0.7190774033016101 0.2733466792329027, axis 0 0 1, limit lower=3.1415 upper=-3.1415 effort=1 velocity=1
- added joint 211_to_110: type revolute, parent 110, child 211, origin xyz=0.21350850196545193 0.8084136149139768 0.715222275585183 rpy=0.2683820677782725 6.282556988648868 1.7771173789542627, axis 1 0 0, limit lower=3.1415 upper=-3.1415 effort=1 velocity=1
- added joint 212_to_110: type revolute, parent 110, child 212, origin xyz=0.21350850196545193 0.8084136149139768 0.715222275585183 rpy=0.4025731016674088 6.282556988648868 1.7771173789542627, axis 1 0 0, limit lower=3.1415 upper=-3.1415 effort=1 velocity=1
- added joint 213_to_110: type revolute, parent 110, child 213, origin xyz=0.21350850196545193 0.8084136149139768 0.715222275585183 rpy=0.536764135556545 6.282556988648868 1.7771173789542627, axis 1 0 0, limit lower=3.1415 upper=-3.1415 effort=1 velocity=1
- added joint 220_to_119: type revolute, parent 119, child 220, origin xyz=0.21350850196545193 0.8084136149139768 0.715222275585183 rpy=0.2683820677782725 6.282556988648868 1.7771173789542627, axis 1 0 0, limit lower=3.1415 upper=-3.1415 effort=1 velocity=1
- added joint 221_to_119: type revolute, parent 119, child 221, origin xyz=0.21350850196545193 0.8084136149139768 0.715222275585183 rpy=0.4025731016674088 6.282556988648868 1.7771173789542627, axis 1 0 0, limit lower=3.1415 upper=-3.1415 effort=1 velocity=1
- added joint 222_to_119: type revolute, parent 119, child 222, origin xyz=0.21350850196545193 0.8084136149139768 0.715222275585183 rpy=0.536764135556545 6.282556988648868 1.7771173789542627, axis 1 0 0, limit lower=3.1415 upper=-3.1415 effort=1 velocity=1
- added joint 22_to_11: type revolute, parent 11, child 22, origin xyz=0.21350850196545193 0.8084136149139768 0.715222275585183 rpy=0.2683820677782725 6.282556988648868 1.7771173789542627, axis 1 0 0, limit lower=3.1415 upper=-3.1415 effort=1 velocity=1
- added joint 23_to_11: type revolute, parent 11, child 23, origin xyz=0.21350850196545193 0.8084136149139768 0.715222275585183 rpy=0.4025731016674088 6.282556988648868 1.7771173789542627, axis 1 0 0, limit lower=3.1415 upper=-3.1415 effort=1 velocity=1
- added joint 24_to_11: type revolute, parent 11, child 24, origin xyz=0.21350850196545193 0.8084136149139768 0.715222275585183 rpy=0.536764135556545 6.282556988648868 1.7771173789542627, axis 1 0 0, limit lower=3.1415 upper=-3.1415 effort=1 velocity=1
- added joint 314_to_110: type revolute, parent 110, child 314, origin xyz=0.1568934003531216 0.1145923753031014 0.993331494039907 rpy=8.271521109969605 3.02010251096389 4.032887921628007, axis 0 0 1, limit lower=3.1415 upper=-3.1415 effort=1 velocity=1
- added joint 315_to_110: type revolute, parent 110, child 315, origin xyz=0.1568934003531216 0.1145923753031014 0.993331494039907 rpy=9.925825331963527 3.02010251096389 4.032887921628007, axis 0 0 1, limit lower=3.1415 upper=-3.1415 effort=1 velocity=1
- added joint 316_to_110: type revolute, parent 110, child 316, origin xyz=0.1568934003531216 0.1145923753031014 0.993331494039907 rpy=11.580129553957446 3.02010251096389 4.032887921628007, axis 0 0 1, limit lower=3.1415 upper=-3.1415 effort=1 velocity=1
- added joint 317_to_110: type revolute, parent 110, child 317, origin xyz=0.1568934003531216 0.1145923753031014 0.993331494039907 rpy=13.234433775951368 3.02010251096389 4.032887921628007, axis 0 0 1, limit lower=3.1415 upper=-3.1415 effort=1 velocity=1
- added joint 318_to_110: type revolute, parent 110, child 318, origin xyz=0.1568934003531216 0.1145923753031014 0.993331494039907 rpy=14.88873799794529 3.02010251096389 4.032887921628007, axis 0 0 1, limit lower=3.1415 upper=-3.1415 effort=1 velocity=1
- added joint 323_to_119: type revolute, parent 119, child 323, origin xyz=0.1568934003531216 0.1145923753031014 0.993331494039907 rpy=8.271521109969605 3.02010251096389 4.032887921628007, axis 0 0 1, limit lower=3.1415 upper=-3.1415 effort=1 velocity=1
- added joint 324_to_119: type revolute, parent 119, child 324, origin xyz=0.1568934003531216 0.1145923753031014 0.993331494039907 rpy=9.925825331963527 3.02010251096389 4.032887921628007, axis 0 0 1, limit lower=3.1415 upper=-3.1415 effort=1 velocity=1
- added joint 325_to_119: type revolute, parent 119, child 325, origin xyz=0.1568934003531216 0.1145923753031014 0.993331494039907 rpy=11.580129553957446 3.02010251096389 4.032887921628007, axis 0 0 1, limit lower=3.1415 upper=-3.1415 effort=1 velocity=1
- added joint 326_to_119: type revolute, parent 119, child 326, origin xyz=0.1568934003531216 0.1145923753031014 0.993331494039907 rpy=13.234433775951368 3.02010251096389 4.032887921628007, axis 0 0 1, limit lower=3.1415 upper=-3.1415 effort=1 velocity=1
- added joint 327_to_119: type revolute, parent 119, child 327, origin xyz=0.1568934003531216 0.1145923753031014 0.993331494039907 rpy=14.88873799794529 3.02010251096389 4.032887921628007, axis 0 0 1, limit lower=3.1415 upper=-3.1415 effort=1 velocity=1
- added joint 35_to_11: type revolute, parent 11, child 35, origin xyz=0.1568934003531216 0.1145923753031014 0.993331494039907 rpy=8.271521109969605 3.02010251096389 4.032887921628007, axis 0 0 1, limit lower=3.1415 upper=-3.1415 effort=1 velocity=1
- added joint 36_to_11: type revolute, parent 11, child 36, origin xyz=0.1568934003531216 0.1145923753031014 0.993331494039907 rpy=9.925825331963527 3.02010251096389 4.032887921628007, axis 0 0 1, limit lower=3.1415 upper=-3.1415 effort=1 velocity=1
- added joint 37_to_11: type revolute, parent 11, child 37, origin xyz=0.1568934003531216 0.1145923753031014 0.993331494039907 rpy=11.580129553957446 3.02010251096389 4.032887921628007, axis 0 0 1, limit lower=3.1415 upper=-3.1415 effort=1 velocity=1
- added joint 38_to_11: type revolute, parent 11, child 38, origin xyz=0.1568934003531216 0.1145923753031014 0.993331494039907 rpy=13.234433775951368 3.02010251096389 4.032887921628007, axis 0 0 1, limit lower=3.1415 upper=-3.1415 effort=1 velocity=1
- added joint 39_to_11: type revolute, parent 11, child 39, origin xyz=0.1568934003531216 0.1145923753031014 0.993331494039907 rpy=14.88873799794529 3.02010251096389 4.032887921628007, axis 0 0 1, limit lower=3.1415 upper=-3.1415 effort=1 velocity=1

File: temp3.urdf (robot description, URDF)
Before this commit: robot pepe, 1 links, 0 joints
Links:
- added link 11, mass 0.08641862943656423; collision cylinder length=1.011626046047713 radius=0.16489927627096637; visual cylinder length=1.011626046047713 radius=0.16489927627096637
- added link 12, mass 0.08641862943656423; collision cylinder length=1.011626046047713 radius=0.16489927627096637; visual cylinder length=1.011626046047713 radius=0.16489927627096637
- added link 13, mass 0.08641862943656423; collision cylinder length=1.011626046047713 radius=0.16489927627096637; visual cylinder length=1.011626046047713 radius=0.16489927627096637
- added link 24, mass 4.858362961097827; collision cylinder length=1.5467743005789663 radius=0.9999; visual cylinder length=1.5467743005789663 radius=0.9999
- added link 25, mass 4.858362961097827; collision cylinder length=1.5467743005789663 radius=0.9999; visual cylinder length=1.5467743005789663 radius=0.9999
- added link 26, mass 4.858362961097827; collision cylinder length=1.5467743005789663 radius=0.9999; visual cylinder length=1.5467743005789663 radius=0.9999
- added link 27, mass 4.858362961097827; collision cylinder length=1.5467743005789663 radius=0.9999; visual cylinder length=1.5467743005789663 radius=0.9999
- link 0: mass 4.666439726850212 -> 0.23124444030073726; geometry collision cylinder length=1.2375544128684464 radius=0.24388133411571777; visual cylinder length=1.2375544128684464 radius=0.24388133411571777
Joints:
- added joint 11_to_0: type revolute, parent 0, child 11, origin xyz=0.21350850196545193 0.7084136149139768 0.615222275585183 rpy=0.2683820677782725 5.944402199549639 1.7771173789542627, axis 0 1 0, limit lower=3.1415 upper=-3.1415 effort=1 velocity=1
- added joint 12_to_0: type revolute, parent 0, child 12, origin xyz=0.21350850196545193 0.7084136149139768 0.615222275585183 rpy=0.4025731016674088 5.944402199549639 1.7771173789542627, axis 0 1 0, limit lower=3.1415 upper=-3.1415 effort=1 velocity=1
- added joint 13_to_0: type revolute, parent 0, child 13, origin xyz=0.21350850196545193 0.7084136149139768 0.615222275585183 rpy=0.536764135556545 5.944402199549639 1.7771173789542627, axis 0 1 0, limit lower=3.1415 upper=-3.1415 effort=1 velocity=1
- added joint 24_to_0: type revolute, parent 0, child 24, origin xyz=0.3746275524862035 0.8223539163707708 0.8441620402522809 rpy=25.46196261499215 4.296523804354824 5.341042113323556, axis 0 1 0, limit lower=3.1415 upper=-3.1415 effort=1 velocity=1
- added joint 25_to_0: type revolute, parent 0, child 25, origin xyz=0.3746275524862035 0.8223539163707708 0.8441620402522809 rpy=30.554355137990576 4.296523804354824 5.341042113323556, axis 0 1 0, limit lower=3.1415 upper=-3.1415 effort=1 velocity=1
- added joint 26_to_0: type revolute, parent 0, child 26, origin xyz=0.3746275524862035 0.8223539163707708 0.8441620402522809 rpy=35.64674766098901 4.296523804354824 5.341042113323556, axis 0 1 0, limit lower=3.1415 upper=-3.1415 effort=1 velocity=1
- added joint 27_to_0: type revolute, parent 0, child 27, origin xyz=0.3746275524862035 0.8223539163707708 0.8441620402522809 rpy=40.73914018398744 4.296523804354824 5.341042113323556, axis 0 1 0, limit lower=3.1415 upper=-3.1415 effort=1 velocity=1

File: temp4.urdf (robot description, URDF)
Before this commit: robot pepe, 4 links, 3 joints
Links:
- link 0: mass 3.4100539802602117 -> 4.858362961097827; geometry collision cylinder length=1.5467743005789663 radius=0.9999; visual cylinder length=1.5467743005789663 radius=0.9999
- link 11: mass 5.922825473440213 -> 0.08641862943656423; geometry collision cylinder length=1.011626046047713 radius=0.16489927627096637; visual cylinder length=1.011626046047713 radius=0.16489927627096637
- link 12: mass 5.922825473440213 -> 0.08641862943656423; geometry collision cylinder length=1.011626046047713 radius=0.16489927627096637; visual cylinder length=1.011626046047713 radius=0.16489927627096637
- link 13: mass 5.922825473440213 -> 0.08641862943656423; geometry collision cylinder length=1.011626046047713 radius=0.16489927627096637; visual cylinder length=1.011626046047713 radius=0.16489927627096637
Joints:
- joint 11_to_0: axis 0 0 1 -> 1 0 0; origin xyz=0.9999 0.9999 0.9999 rpy=8.943082072563138 6.282556988648868 6.282556988648868 -> xyz=0.11350850196545192 0.7084136149139768 0.715222275585183 rpy=1.52501912921419 5.944402199549639 3.0337544403901795
- joint 12_to_0: axis 0 0 1 -> 1 0 0; origin xyz=0.9999 0.9999 0.9999 rpy=13.414623108844708 6.282556988648868 6.282556988648868 -> xyz=0.11350850196545192 0.7084136149139768 0.715222275585183 rpy=2.287528693821285 5.944402199549639 3.0337544403901795
- joint 13_to_0: axis 0 0 1 -> 1 0 0; origin xyz=0.9999 0.9999 0.9999 rpy=17.886164145126276 6.282556988648868 6.282556988648868 -> xyz=0.11350850196545192 0.7084136149139768 0.715222275585183 rpy=3.05003825842838 5.944402199549639 3.0337544403901795

File: temp5.urdf (robot description, URDF)
Before this commit: robot pepe, 4 links, 3 joints
Links:
- added link 14, mass 4.858362961097827; collision cylinder length=1.5467743005789663 radius=0.9999; visual cylinder length=1.5467743005789663 radius=0.9999
- link 0: mass 3.4100539802602117 -> 4.858362961097827; geometry collision cylinder length=1.5467743005789663 radius=0.9999; visual cylinder length=1.5467743005789663 radius=0.9999
- link 11: mass 5.922825473440213 -> 4.858362961097827; geometry collision cylinder length=1.5467743005789663 radius=0.9999; visual cylinder length=1.5467743005789663 radius=0.9999
- link 12: mass 5.922825473440213 -> 4.858362961097827; geometry collision cylinder length=1.5467743005789663 radius=0.9999; visual cylinder length=1.5467743005789663 radius=0.9999
- link 13: mass 5.922825473440213 -> 4.858362961097827; geometry collision cylinder length=1.5467743005789663 radius=0.9999; visual cylinder length=1.5467743005789663 radius=0.9999
Joints:
- added joint 14_to_0: type revolute, parent 0, child 14, origin xyz=0.3746275524862035 0.9223539163707708 0.8441620402522809 rpy=25.46196261499215 4.296523804354824 5.341042113323556, axis 0 1 0, limit lower=3.1415 upper=-3.1415 effort=1 velocity=1
- joint 11_to_0: axis 0 0 1 -> 0 1 0; origin xyz=0.9999 0.9999 0.9999 rpy=8.943082072563138 6.282556988648868 6.282556988648868 -> xyz=0.3746275524862035 0.9223539163707708 0.8441620402522809 rpy=10.18478504599686 4.296523804354824 5.341042113323556
- joint 12_to_0: axis 0 0 1 -> 0 1 0; origin xyz=0.9999 0.9999 0.9999 rpy=13.414623108844708 6.282556988648868 6.282556988648868 -> xyz=0.3746275524862035 0.9223539163707708 0.8441620402522809 rpy=15.277177568995288 4.296523804354824 5.341042113323556
- joint 13_to_0: axis 0 0 1 -> 0 1 0; origin xyz=0.9999 0.9999 0.9999 rpy=17.886164145126276 6.282556988648868 6.282556988648868 -> xyz=0.3746275524862035 0.9223539163707708 0.8441620402522809 rpy=20.36957009199372 4.296523804354824 5.341042113323556
