Commit message: genome spec experiments

File: temp6.urdf (robot description, URDF)
Before this commit: robot pepe, 4 links, 3 joints
Links:
- added link 14, mass 5.486555834392827; collision cylinder length=1.7467743005789662 radius=0.9999; visual cylinder length=1.7467743005789662 radius=0.9999
- link 0: mass 3.4100539802602117 -> 0.22301363611944708; geometry collision cylinder length=1.011626046047713 radius=0.2648992762709664; visual cylinder length=1.011626046047713 radius=0.2648992762709664
- link 11: mass 4.038246853555211 -> 5.486555834392827; geometry collision cylinder length=1.7467743005789662 radius=0.9999; visual cylinder length=1.7467743005789662 radius=0.9999
- link 12: mass 4.038246853555211 -> 5.486555834392827; geometry collision cylinder length=1.7467743005789662 radius=0.9999; visual cylinder length=1.7467743005789662 radius=0.9999
- link 13: mass 4.038246853555211 -> 5.486555834392827; geometry collision cylinder length=1.7467743005789662 radius=0.9999; visual cylinder length=1.7467743005789662 radius=0.9999
Joints:
- added joint 14_to_0: type revolute, parent 0, child 14, origin xyz=0.3746275524862035 0.8223539163707708 0.9441620402522809 rpy=25.46196261499215 4.296523804354824 5.969360644041514, axis 0 1 0, limit lower=3.1415 upper=-3.1415 effort=1 velocity=1
- joint 11_to_0: axis 0 0 1 -> 0 1 0; origin xyz=0.9999 0.9500845945394578 0.9999 rpy=6.4298079496913045 3.8001087162635065 5.976593086836112 -> xyz=0.3746275524862035 0.8223539163707708 0.9441620402522809 rpy=10.18478504599686 4.296523804354824 5.969360644041514
- joint 12_to_0: axis 0 0 1 -> 0 1 0; origin xyz=0.9999 0.9500845945394578 0.9999 rpy=9.644711924536956 3.8001087162635065 5.976593086836112 -> xyz=0.3746275524862035 0.8223539163707708 0.9441620402522809 rpy=15.277177568995288 4.296523804354824 5.969360644041514
- joint 13_to_0: axis 0 0 1 -> 0 1 0; origin xyz=0.9999 0.9500845945394578 0.9999 rpy=12.859615899382609 3.8001087162635065 5.976593086836112 -> xyz=0.3746275524862035 0.8223539163707708 0.9441620402522809 rpy=20.36957009199372 4.296523804354824 5.969360644041514

File: temp7.urdf (robot description, URDF)
Before this commit: robot pepe, 4 links, 3 joints
Links:
- link 0: mass 5.922825473440213 -> 4.858362961097827; geometry collision cylinder length=1.5467743005789663 radius=0.9999; visual cylinder length=1.5467743005789663 radius=0.9999
- link 11: mass 0.4203795558477106 -> 0.08641862943656423; geometry collision cylinder length=1.011626046047713 radius=0.16489927627096637; visual cylinder length=1.011626046047713 radius=0.16489927627096637
- link 12: mass 0.4203795558477106 -> 0.08641862943656423; geometry collision cylinder length=1.011626046047713 radius=0.16489927627096637; visual cylinder length=1.011626046047713 radius=0.16489927627096637
- link 13: mass 0.4203795558477106 -> 0.08641862943656423; geometry collision cylinder length=1.011626046047713 radius=0.16489927627096637; visual cylinder length=1.011626046047713 radius=0.16489927627096637
Joints:
- joint 11_to_0: axis 0 0 1 -> 1 0 0; origin xyz=0.5507040907358064 0.5018865040146698 0.48089488158635463 rpy=12.565113977297736 6.282556988648868 5.352476816319871 -> xyz=0.11350850196545192 0.7084136149139768 0.5152222755851831 rpy=0.2683820677782725 6.282556988648868 2.405435909672221
- joint 12_to_0: axis 0 0 1 -> 1 0 0; origin xyz=0.5507040907358064 0.5018865040146698 0.48089488158635463 rpy=18.847670965946605 6.282556988648868 5.352476816319871 -> xyz=0.11350850196545192 0.7084136149139768 0.5152222755851831 rpy=0.4025731016674088 6.282556988648868 2.405435909672221
- joint 13_to_0: axis 0 0 1 -> 1 0 0; origin xyz=0.5507040907358064 0.5018865040146698 0.48089488158635463 rpy=25.130227954595473 6.282556988648868 5.352476816319871 -> xyz=0.11350850196545192 0.7084136149139768 0.5152222755851831 rpy=0.536764135556545 6.282556988648868 2.405435909672221

File: test.urdf (robot description, URDF)
Before this commit: robot pepe, 6 links, 5 joints
Links:
- removed link 13
- removed link 14
- removed link 15
- added link 23, mass 0.07963559138428422; collision cylinder length=0.7012565373454558 radius=0.19012542898013365; visual cylinder length=0.7012565373454558 radius=0.19012542898013365
- added link 24, mass 0.07963559138428422; collision cylinder length=0.7012565373454558 radius=0.19012542898013365; visual cylinder length=0.7012565373454558 radius=0.19012542898013365
- added link 25, mass 0.07963559138428422; collision cylinder length=0.7012565373454558 radius=0.19012542898013365; visual cylinder length=0.7012565373454558 radius=0.19012542898013365
- link 0: mass 0.08641862943656423 -> 0.1419061211900836; geometry collision cylinder length=0.28565514550564536 radius=0.3976533107610025; visual cylinder length=0.28565514550564536 radius=0.3976533107610025
- link 11: mass 1.6909907427759374 -> 0.42613922069035665; geometry collision cylinder length=0.13567145977163642 radius=0.9999; visual cylinder length=0.13567145977163642 radius=0.9999
- link 12: mass 1.6909907427759374 -> 0.42613922069035665; geometry collision cylinder length=0.13567145977163642 radius=0.9999; visual cylinder length=0.13567145977163642 radius=0.9999
Joints:
- removed joint 13_to_0
- removed joint 14_to_0
- removed joint 15_to_0
- added joint 23_to_0: type revolute, parent 0, child 23, origin xyz=0.6844122646964637 0.9604018281320923 0.7728727567543932 rpy=22.800443265250202 3.009560276144289 4.5452777247438085, axis 0 1 0, limit lower=3.1415 upper=-3.1415 effort=1 velocity=1
- added joint 24_to_0: type revolute, parent 0, child 24, origin xyz=0.6844122646964637 0.9604018281320923 0.7728727567543932 rpy=28.500554081562754 3.009560276144289 4.5452777247438085, axis 0 1 0, limit lower=3.1415 upper=-3.1415 effort=1 velocity=1
- added joint 25_to_0: type revolute, parent 0, child 25, origin xyz=0.6844122646964637 0.9604018281320923 0.7728727567543932 rpy=34.2006648978753 3.009560276144289 4.5452777247438085, axis 0 1 0, limit lower=3.1415 upper=-3.1415 effort=1 velocity=1
- joint 11_to_0: axis 0 1 0 -> 0 0 1; origin xyz=0.5457165619257499 0.2359593594716205 0.8315587841570061 rpy=11.401585670435251 2.863602954693267 3.9043382821833372 -> xyz=0.7687475341915667 0.9999 0.13073779713381786 rpy=5.480410577574733 3.73896713734325 0.09024802037923292
- joint 12_to_0: axis 0 1 0 -> 0 0 1; origin xyz=0.5457165619257499 0.2359593594716205 0.8315587841570061 rpy=17.102378505652876 2.863602954693267 3.9043382821833372 -> xyz=0.7687475341915667 0.9999 0.13073779713381786 rpy=8.220615866362099 3.73896713734325 0.09024802037923292
